File: TRX055.01.01.PB.00.00/TRX055.01.01.PB.00.00.kicad_pcb (KiCad board)
At the start: 4 copper layers, 91.3 x 139.8 mm, 143 parts, among them J1 DF40HC-80DS, J2 DF40HC-80DS, J3 DF40HC-80DS, J4 DF40HC-80DS, U1 XC7Z015-1CLG485I, U2 AS4C256M16D3, U3 AS4C256M16D3, U5 AP22913CN4, U9 AP22913CN4

Commit message: Update Layout
Parts:
- removed FB1, FB2, FB3, FB4, FB5: FerriteBead, Inductor_SMD:L_0603_1608Metric
- added C108: M1, Capacitor_SMD:C_0402_1005Metric, F.Cu at (139.0, 71.8)
- added C109: M1, Capacitor_SMD:C_0402_1005Metric, F.Cu at (138.0, 71.8)
- added C110: M1, Capacitor_SMD:C_0402_1005Metric, F.Cu at (142.5, 71.9)
- added C111: M1, Capacitor_SMD:C_0402_1005Metric, F.Cu at (143.6, 71.9)
- added FL1: Choke_Schaffner_RN102-0.3-02-12M, Inductor_THT:Choke_Schaffner_RN102-04-14.0x14.0mm, F.Cu at (175.0, 115.5)
- added J5: SFP, Connector:Connector_SFP_and_Cage, F.Cu at (141.0, 68.7)
- added J6: Micro_SD_Card, Connector_Card:microSD_HC_Molex_47219-2001, B.Cu at (69.9, 61.7)
- added R12: 33R, Resistor_SMD:R_0402_1005Metric, F.Cu at (79.2, 74.8)
- added R14: 33R, Resistor_SMD:R_0402_1005Metric, F.Cu at (79.2, 73.8)
- added R17: 33R, Resistor_SMD:R_0402_1005Metric, F.Cu at (79.2, 76.7)
- added R18: 33R, Resistor_SMD:R_0402_1005Metric, F.Cu at (79.2, 79.5)
- added R19: 33R, Resistor_SMD:R_0402_1005Metric, F.Cu at (79.2, 81.5)
- added R20: 33R, Resistor_SMD:R_0402_1005Metric, F.Cu at (79.2, 75.8)
- added R21: 33R, Resistor_SMD:R_0402_1005Metric, F.Cu at (79.2, 80.5)
- added R22: 33R, Resistor_SMD:R_0402_1005Metric, F.Cu at (79.2, 77.7)
- added R23: 33R, Resistor_SMD:R_0402_1005Metric, F.Cu at (79.2, 82.4)
- added R24: 33R, Resistor_SMD:R_0402_1005Metric, F.Cu at (79.2, 83.3)
- added R25: 33R, Resistor_SMD:R_0402_1005Metric, F.Cu at (79.2, 84.3)
- added R26: 33R, Resistor_SMD:R_0402_1005Metric, F.Cu at (79.2, 78.6)
- added R27: 33R, Resistor_SMD:R_0402_1005Metric, F.Cu at (77.6, 87.9)
- added R28: 33R, Resistor_SMD:R_0402_1005Metric, F.Cu at (76.4, 86.5)
- added R29: 33R, Resistor_SMD:R_0402_1005Metric, F.Cu at (74.6, 74.0)
- added U10: ~, ppa-active:XQFN16, F.Cu at (86.5, 75.0)
- added U11: KSZ9031RNXCA, Package_DFN_QFN:QFN-48-1EP_7x7mm_P0.5mm_EP5.15x5.15mm, F.Cu at (82.7, 51.8)
- added U12: USB3320C-EZK-TR, Package_DFN_QFN:QFN-32-1EP_5x5mm_P0.5mm_EP3.3x3.3mm, F.Cu at (71.0, 81.6)
- added U14: W25Q128JVSIQ, Package_SO:SOIC-8_5.23x5.23mm_P1.27mm, F.Cu at (83.0, 70.2)
- U2, U3: value AS4C256M16D3 -> K4B4G1646E-BYMA
- moved J4 97.8 mm to (83.0, 138.0), turned to 0 degrees
- moved J1 90.9 mm to (128.0, 93.0), turned to 180 degrees
- moved C85 68.2 mm to (160.5, 87.0)
- moved J2 34.8 mm to (128.0, 138.0)
- moved J3 27.7 mm to (83.0, 93.0)
- moved U9 27.0 mm to (93.4, 95.9)
- moved U5 27.0 mm to (97.0, 96.0)
- moved C100 24.3 mm to (127.8, 62.7), turned to -90 degrees
- moved C97 23.4 mm to (127.2, 62.7), turned to -90 degrees
- moved C88 23.1 mm to (139.2, 74.0)
- moved C92 23.1 mm to (139.2, 74.7)
- moved C45 22.1 mm to (104.8, 92.4)
- moved C93 19.7 mm to (126.2, 62.7), turned to -90 degrees
- moved C89 18.8 mm to (125.5, 62.7), turned to -90 degrees
- moved C107 15.0 mm to (109.7, 89.9), turned to 90 degrees
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Connections:
- C100 pad 1: unconnected-(C100-Pad1) -> /GT_TX2_N
- C100 pad 2: Net-(U1A-MGTPTXP1_112) -> Net-(U1J-MGTPTXN2_112)
- C101 pad 1: unconnected-(C101-Pad1) -> /GT_TX2_P
- C101 pad 2: Net-(U1A-MGTPTXP0_112) -> Net-(U1J-MGTPTXP2_112)
- C102 pad 1: unconnected-(C102-Pad1) -> /GT_TX3_N
- C102 pad 2: Net-(U1A-MGTPTXP3_112) -> Net-(U1J-MGTPTXN3_112)
- C103 pad 1: unconnected-(C103-Pad1) -> /GT_TX3_P
- C103 pad 2: Net-(U1A-MGTPTXP2_112) -> Net-(U1J-MGTPTXP3_112)
- C104 pad 1: unconnected-(C104-Pad1) -> /GTP_REF_CLK0_P
- C104 pad 2: Net-(U1A-MGTREFCLK0N_112) -> Net-(U1J-MGTREFCLK0P_112)
- C105 pad 1: unconnected-(C105-Pad1) -> /GTP_REF_CLK1_N
- C105 pad 2: Net-(U1A-MGTREFCLK1N_112) -> Net-(U1J-MGTREFCLK1P_112)
- C106 pad 1: unconnected-(C106-Pad1) -> /GTP_REF_CLK0_N
- C106 pad 2: Net-(U1A-MGTREFCLK0P_112) -> Net-(U1J-MGTREFCLK0N_112)
- C107 pad 1: unconnected-(C107-Pad1) -> /GTP_REF_CLK1_P
- C107 pad 2: Net-(U1A-MGTREFCLK1P_112) -> Net-(U1J-MGTREFCLK1N_112)
- C28 pad 1: /ZynqPower/VCCINT -> /ZynqPower/1V_RAIL_B
- C29 pad 1: /ZynqPower/VCCINT -> /ZynqPower/1V_RAIL_B
- C30 pad 1: /ZynqPower/VCCINT -> /ZynqPower/1V_RAIL_B
- C31 pad 1: /ZynqPower/VCCINT -> /ZynqPower/1V_RAIL_B
- C32 pad 1: /ZynqPower/VCCINT -> /ZynqPower/1V_RAIL_B
- C33 pad 1: /ZynqPower/VCCINT -> /ZynqPower/1V_RAIL_B
- C34 pad 1: /ZynqPower/VCCINT -> /ZynqPower/1V_RAIL_B
- C35 pad 1: /ZynqPower/VCCINT -> /ZynqPower/1V_RAIL_B
- C36 pad 1: /ZynqPower/VCCAUX -> VCC_MIO
- C37 pad 1: /ZynqPower/VCCAUX -> VCC_MIO
- C38 pad 1: /ZynqPower/VCCAUX -> VCC_MIO
- C39 pad 1: /ZynqPower/VCCAUX -> VCC_MIO
- C51 pad 1: /ZynqPower/PS_CORE -> /ZynqPower/1V_RAIL_A
- C52 pad 1: /ZynqPower/PS_CORE -> /ZynqPower/1V_RAIL_A
- C53 pad 1: /ZynqPower/PS_CORE -> /ZynqPower/1V_RAIL_A
- C54 pad 1: /ZynqPower/PS_CORE -> /ZynqPower/1V_RAIL_A
- C55 pad 1: /ZynqPower/PS_CORE -> /ZynqPower/1V_RAIL_A
- C56 pad 1: /ZynqPower/PS_CORE -> /ZynqPower/1V_RAIL_A
- C57 pad 1: /ZynqPower/VCCPAUX -> /ZynqPower/1V8_RAIL_A
- C58 pad 1: /ZynqPower/VCCPAUX -> /ZynqPower/1V8_RAIL_A
- C59 pad 1: /ZynqPower/VCCPAUX -> /ZynqPower/1V8_RAIL_A
- C60 pad 1: /ZynqPower/VCCPAUX -> /ZynqPower/1V8_RAIL_A
- C88 pad 1: unconnected-(C88-Pad1) -> /GT_RX1_P
- C88 pad 2: Net-(U1A-MGTPRXN0_112) -> Net-(U1J-MGTPRXP1_112)
- C89 pad 1: unconnected-(C89-Pad1) -> /GT_RX1_N
- C90 pad 1: unconnected-(C90-Pad1) -> /GT_RX0_P
- C90 pad 2: Net-(U1A-MGTPRXN2_112) -> Net-(U1J-MGTPRXP0_112)
- C91 pad 1: unconnected-(C91-Pad1) -> /GT_RX0_N
- C91 pad 2: Net-(U1A-MGTPRXN3_112) -> Net-(U1J-MGTPRXN0_112)
- C92 pad 1: unconnected-(C92-Pad1) -> /GT_RX2_P
- C92 pad 2: Net-(U1A-MGTPRXP0_112) -> Net-(U1J-MGTPRXP2_112)
- C93 pad 1: unconnected-(C93-Pad1) -> /GT_RX2_N
- C93 pad 2: Net-(U1A-MGTPRXP1_112) -> Net-(U1J-MGTPRXN2_112)
- C94 pad 1: unconnected-(C94-Pad1) -> /GT_RX3_P
- C94 pad 2: Net-(U1A-MGTPRXP2_112) -> Net-(U1J-MGTPRXP3_112)
- C95 pad 1: unconnected-(C95-Pad1) -> /GT_RX3_N
- C95 pad 2: Net-(U1A-MGTPRXP3_112) -> Net-(U1J-MGTPRXN3_112)
- C96 pad 1: unconnected-(C96-Pad1) -> /GT_TX0_P
- C96 pad 2: Net-(U1A-MGTPTXN0_112) -> Net-(U1J-MGTPTXP0_112)
- C97 pad 1: unconnected-(C97-Pad1) -> /GT_TX0_N
- C97 pad 2: Net-(U1A-MGTPTXN1_112) -> Net-(U1J-MGTPTXN0_112)
- C98 pad 1: unconnected-(C98-Pad1) -> /GT_TX1_N
- C98 pad 2: Net-(U1A-MGTPTXN3_112) -> Net-(U1J-MGTPTXN1_112)
- C99 pad 1: unconnected-(C99-Pad1) -> /GT_TX1_P
- C99 pad 2: Net-(U1A-MGTPTXN2_112) -> Net-(U1J-MGTPTXP1_112)
- FB11 pad 1: Net-(U5-OUT) -> VCC_MIO
- J1 pad 1: /Module_A1/MOD_SPI_MOSI -> VDD_5V5A
- J1 pad 10: VDD_SYSTEM -> unconnected-(J1-Pad10)
- J1 pad 11: /Module_A1/LS_GPIO2 -> Net-(J1-Pad11)
- J1 pad 12: GND -> unconnected-(J1-Pad12)
- J1 pad 13: /Module_A1/LS_GPIO3 -> GND
- J1 pad 14: VDD_5V5A -> /Module_A1/HS_VREF
- J1 pad 15: /Module_A1/LS_GPIO4 -> Net-(J1-Pad15)
- J1 pad 16: VDD_5V5A -> unconnected-(J1-Pad16)
- J1 pad 17: /Module_A1/LS_GPIO5 -> GND
- J1 pad 18: VDD_5V5A -> GND
- J1 pad 19: /Module_A1/LS_GPIO6 -> /GTP_REF_CLK1_P
- J1 pad 20: GND -> /Module_A1/HS_DIFF_CLK1_P
- J1 pad 21: /Module_A1/LS_GPIO7 -> /GTP_REF_CLK1_N
- J1 pad 22: GND -> /Module_A1/HS_DIFF_CLK1_N
- J1 pad 23: /Module_A1/LS_GPIO8 -> GND
- J1 pad 24: VDD_3V3D -> GND
- J1 pad 25: /Module_A1/LS_GPIO9 -> /GT_TX3_N
- J1 pad 26: VDD_3V3D -> /GT_RX3_N
- J1 pad 27: GND -> /GT_TX3_P
- J1 pad 28: VDD_1V8D -> /GT_RX3_P
- J1 pad 29: Net-(J1-Pad29) -> /GT_TX2_N
- J1 pad 3: /Module_A1/MOD_SPI_MISO -> VDD_5V5A
- J1 pad 30: /Module_A1/LS_VREF -> /GT_RX2_N
- J1 pad 31: GND -> /GT_TX2_P
- J1 pad 32: /Module_A1/HS_VREF -> /GT_RX2_P
- J1 pad 33: Net-(J1-Pad33) -> GND
- J1 pad 35: /Module_A1/HS_DIFF_CLK1_N -> /Module_A1/HS_DIFF_5_N
- J1 pad 36: /Module_A1/HS_DIFF_CLK0_N -> /Module_A1/HS_DIFF_4_N
- J1 pad 37: /Module_A1/HS_DIFF_CLK1_P -> /Module_A1/HS_DIFF_5_P
- J1 pad 38: /Module_A1/HS_DIFF_CLK0_P -> /Module_A1/HS_DIFF_4_P
- J1 pad 39: GND -> /Module_A1/HS_DIFF_7_N
- J1 pad 40: GND -> /Module_A1/HS_DIFF_6_N
- J1 pad 41: /Module_A1/HS_DIFF_15_N -> /Module_A1/HS_DIFF_7_P
- J1 pad 42: /Module_A1/HS_DIFF_7_N -> /Module_A1/HS_DIFF_6_P
- J1 pad 43: /Module_A1/HS_DIFF_15_P -> /Module_A1/HS_DIFF_9_N
- J1 pad 44: /Module_A1/HS_DIFF_7_P -> /Module_A1/HS_DIFF_8_N
- J1 pad 45: /Module_A1/HS_DIFF_14_N -> /Module_A1/HS_DIFF_9_P
- J1 pad 46: /Module_A1/HS_DIFF_6_N -> /Module_A1/HS_DIFF_8_P
- J1 pad 47: /Module_A1/HS_DIFF_14_P -> GND
- J1 pad 48: /Module_A1/HS_DIFF_6_P -> GND
- J1 pad 49: GND -> /Module_A1/HS_DIFF_11_N
- J1 pad 5: /Module_A1/MOD_SPI_SCK -> VDD_3V3D
- J1 pad 50: GND -> /Module_A1/HS_DIFF_10_N
- J1 pad 51: /Module_A1/HS_DIFF_13_N -> /Module_A1/HS_DIFF_11_P
- J1 pad 52: /Module_A1/HS_DIFF_5_N -> /Module_A1/HS_DIFF_10_P
- J1 pad 53: /Module_A1/HS_DIFF_13_P -> /Module_A1/HS_DIFF_13_N
- J1 pad 54: /Module_A1/HS_DIFF_5_P -> /Module_A1/HS_DIFF_12_N
- J1 pad 55: /Module_A1/HS_DIFF_12_N -> /Module_A1/HS_DIFF_13_P
- J1 pad 56: /Module_A1/HS_DIFF_4_N -> /Module_A1/HS_DIFF_12_P
- J1 pad 57: /Module_A1/HS_DIFF_12_P -> /Module_A1/HS_DIFF_15_N
- J1 pad 58: /Module_A1/HS_DIFF_4_P -> /Module_A1/HS_DIFF_14_N
- J1 pad 59: GND -> /Module_A1/HS_DIFF_15_P
- J1 pad 60: GND -> /Module_A1/HS_DIFF_14_P
- J1 pad 61: /Module_A1/HS_DIFF_11_N -> GND
- J1 pad 62: /Module_A1/HS_DIFF_3_N -> GND
- J1 pad 63: /Module_A1/HS_DIFF_11_P -> /Module_A1/LS_GPIO4
- J1 pad 64: /Module_A1/HS_DIFF_3_P -> /Module_A1/LS_VREF
- J1 pad 65: /Module_A1/HS_DIFF_10_N -> /Module_A1/LS_GPIO5
- J1 pad 66: /Module_A1/HS_DIFF_2_N -> /Module_A1/MOD_SPI_SCK
- J1 pad 67: /Module_A1/HS_DIFF_10_P -> /Module_A1/LS_GPIO6
- J1 pad 68: /Module_A1/HS_DIFF_2_P -> /Module_A1/MOD_SPI_MISO
- J1 pad 69: GND -> /Module_A1/I2C_A2
- J1 pad 7: /Module_A1/LS_GPIO0 -> VDD_3V3D
- J1 pad 70: GND -> /Module_A1/MOD_SPI_MOSI
- J1 pad 71: /Module_A1/HS_DIFF_9_N -> /Module_A1/I2C_A1
- J1 pad 72: /Module_A1/HS_DIFF_1_N -> /Module_A1/LS_GPIO0
- J1 pad 73: /Module_A1/HS_DIFF_9_P -> /Module_A1/I2C_A0
- J1 pad 74: /Module_A1/HS_DIFF_1_P -> /Module_A1/LS_GPIO1
- J1 pad 75: /Module_A1/HS_DIFF_8_N -> /Module_A1/I2C_SDA
- J1 pad 76: /Module_A1/HS_DIFF_0_N -> /Module_A1/LS_GPIO2
- J1 pad 77: /Module_A1/HS_DIFF_8_P -> /Module_A1/I2C_SCL
- J1 pad 78: /Module_A1/HS_DIFF_0_P -> /Module_A1/LS_GPIO3
- J1 pad 8: VDD_SYSTEM -> VDD_1V8D
- J1 pad 9: /Module_A1/LS_GPIO1 -> GND
- J2 pad 1: /Module_A2/MOD_SPI_MOSI -> VDD_5V5A
- J2 pad 10: VDD_SYSTEM -> unconnected-(J2-Pad10)
- J2 pad 11: /Module_A2/LS_GPIO2 -> Net-(J2-Pad11)
- J2 pad 12: GND -> unconnected-(J2-Pad12)
- J2 pad 13: /Module_A2/LS_GPIO3 -> GND
- J2 pad 14: VDD_5V5A -> /Module_A2/HS_VREF
- J2 pad 15: /Module_A2/LS_GPIO4 -> Net-(J2-Pad15)
- J2 pad 16: VDD_5V5A -> unconnected-(J2-Pad16)
- J2 pad 17: /Module_A2/LS_GPIO5 -> GND
- J2 pad 18: VDD_5V5A -> GND
- J2 pad 19: /Module_A2/LS_GPIO6 -> /Module_A2/HS_DIFF_CLK0_P
- J2 pad 20: GND -> /Module_A2/HS_DIFF_CLK1_P
- J2 pad 21: /Module_A2/LS_GPIO7 -> /Module_A2/HS_DIFF_CLK0_N
- J2 pad 22: GND -> /Module_A2/HS_DIFF_CLK1_N
- J2 pad 23: /Module_A2/LS_GPIO8 -> GND
- J2 pad 24: VDD_3V3D -> GND
- J2 pad 25: /Module_A2/LS_GPIO9 -> /Module_A2/HS_DIFF_1_N
- J2 pad 26: VDD_3V3D -> /Module_A2/HS_DIFF_0_N
- J2 pad 27: GND -> /Module_A2/HS_DIFF_1_P
- J2 pad 28: VDD_1V8D -> /Module_A2/HS_DIFF_0_P
- J2 pad 29: Net-(J2-Pad29) -> /Module_A2/HS_DIFF_3_N
- J2 pad 3: /Module_A2/MOD_SPI_MISO -> VDD_5V5A
- J2 pad 30: /Module_A2/LS_VREF -> /Module_A2/HS_DIFF_2_N
- J2 pad 31: GND -> /Module_A2/HS_DIFF_3_P
- J2 pad 32: /Module_A2/HS_VREF -> /Module_A2/HS_DIFF_2_P
- J2 pad 33: Net-(J2-Pad33) -> GND
- J2 pad 35: /Module_A2/HS_DIFF_CLK1_N -> /Module_A2/HS_DIFF_5_N
- J2 pad 36: /Module_A2/HS_DIFF_CLK0_N -> /Module_A2/HS_DIFF_4_N
- J2 pad 37: /Module_A2/HS_DIFF_CLK1_P -> /Module_A2/HS_DIFF_5_P
- J2 pad 38: /Module_A2/HS_DIFF_CLK0_P -> /Module_A2/HS_DIFF_4_P
- J2 pad 39: GND -> /Module_A2/HS_DIFF_7_N
- J2 pad 40: GND -> /Module_A2/HS_DIFF_6_N
- J2 pad 41: /Module_A2/HS_DIFF_15_N -> /Module_A2/HS_DIFF_7_P
- J2 pad 42: /Module_A2/HS_DIFF_7_N -> /Module_A2/HS_DIFF_6_P
- J2 pad 43: /Module_A2/HS_DIFF_15_P -> /Module_A2/HS_DIFF_9_N
- J2 pad 44: /Module_A2/HS_DIFF_7_P -> /Module_A2/HS_DIFF_8_N
- J2 pad 45: /Module_A2/HS_DIFF_14_N -> /Module_A2/HS_DIFF_9_P
- J2 pad 46: /Module_A2/HS_DIFF_6_N -> /Module_A2/HS_DIFF_8_P
- J2 pad 47: /Module_A2/HS_DIFF_14_P -> GND
- J2 pad 48: /Module_A2/HS_DIFF_6_P -> GND
- J2 pad 49: GND -> /Module_A2/HS_DIFF_11_N
- J2 pad 5: /Module_A2/MOD_SPI_SCK -> VDD_3V3D
- J2 pad 50: GND -> /Module_A2/HS_DIFF_10_N
- J2 pad 51: /Module_A2/HS_DIFF_13_N -> /Module_A2/HS_DIFF_11_P
- J2 pad 52: /Module_A2/HS_DIFF_5_N -> /Module_A2/HS_DIFF_10_P
- J2 pad 53: /Module_A2/HS_DIFF_13_P -> /Module_A2/HS_DIFF_13_N
- J2 pad 54: /Module_A2/HS_DIFF_5_P -> /Module_A2/HS_DIFF_12_N
- J2 pad 55: /Module_A2/HS_DIFF_12_N -> /Module_A2/HS_DIFF_13_P
- J2 pad 56: /Module_A2/HS_DIFF_4_N -> /Module_A2/HS_DIFF_12_P
- J2 pad 57: /Module_A2/HS_DIFF_12_P -> /Module_A2/HS_DIFF_15_N
- J2 pad 58: /Module_A2/HS_DIFF_4_P -> /Module_A2/HS_DIFF_14_N
- J2 pad 59: GND -> /Module_A2/HS_DIFF_15_P
- J2 pad 60: GND -> /Module_A2/HS_DIFF_14_P
- J2 pad 61: /Module_A2/HS_DIFF_11_N -> GND
- J2 pad 62: /Module_A2/HS_DIFF_3_N -> GND
- J2 pad 63: /Module_A2/HS_DIFF_11_P -> /Module_A2/LS_GPIO4
- J2 pad 64: /Module_A2/HS_DIFF_3_P -> /Module_A2/LS_VREF
- J2 pad 65: /Module_A2/HS_DIFF_10_N -> /Module_A2/LS_GPIO5
- J2 pad 66: /Module_A2/HS_DIFF_2_N -> /Module_A2/MOD_SPI_SCK
- J2 pad 67: /Module_A2/HS_DIFF_10_P -> /Module_A2/LS_GPIO6
- J2 pad 68: /Module_A2/HS_DIFF_2_P -> /Module_A2/MOD_SPI_MISO
- J2 pad 69: GND -> /Module_A2/I2C_A2
- J2 pad 7: /Module_A2/LS_GPIO0 -> VDD_3V3D
- J2 pad 70: GND -> /Module_A2/MOD_SPI_MOSI
- J2 pad 71: /Module_A2/HS_DIFF_9_N -> /Module_A2/I2C_A1
- J2 pad 72: /Module_A2/HS_DIFF_1_N -> /Module_A2/LS_GPIO0
- J2 pad 73: /Module_A2/HS_DIFF_9_P -> /Module_A2/I2C_A0
- J2 pad 74: /Module_A2/HS_DIFF_1_P -> /Module_A2/LS_GPIO1
- J2 pad 75: /Module_A2/HS_DIFF_8_N -> /Module_A2/I2C_SDA
- J2 pad 76: /Module_A2/HS_DIFF_0_N -> /Module_A2/LS_GPIO2
- J2 pad 77: /Module_A2/HS_DIFF_8_P -> /Module_A2/I2C_SCL
- J2 pad 78: /Module_A2/HS_DIFF_0_P -> /Module_A2/LS_GPIO3
- J2 pad 8: VDD_SYSTEM -> VDD_1V8D
- J2 pad 9: /Module_A2/LS_GPIO1 -> GND
- J3 pad 1: /Module_A3/MOD_SPI_MOSI -> VDD_5V5A
- J3 pad 10: VDD_SYSTEM -> unconnected-(J3-Pad10)
- J3 pad 11: /Module_A3/LS_GPIO2 -> Net-(J3-Pad11)
- J3 pad 12: GND -> unconnected-(J3-Pad12)
- J3 pad 13: /Module_A3/LS_GPIO3 -> GND
- J3 pad 14: VDD_5V5A -> /Module_A3/HS_VREF
- J3 pad 15: /Module_A3/LS_GPIO4 -> Net-(J3-Pad15)
- J3 pad 16: VDD_5V5A -> unconnected-(J3-Pad16)
- J3 pad 17: /Module_A3/LS_GPIO5 -> GND
- J3 pad 18: VDD_5V5A -> GND
- J3 pad 19: /Module_A3/LS_GPIO6 -> /Module_A3/HS_DIFF_CLK0_P
- J3 pad 20: GND -> /Module_A3/HS_DIFF_CLK1_P
- J3 pad 21: /Module_A3/LS_GPIO7 -> /Module_A3/HS_DIFF_CLK0_N
- J3 pad 22: GND -> /Module_A3/HS_DIFF_CLK1_N
- J3 pad 23: /Module_A3/LS_GPIO8 -> GND
- J3 pad 24: VDD_3V3D -> GND
- J3 pad 25: /Module_A3/LS_GPIO9 -> /Module_A3/HS_DIFF_1_N
- J3 pad 26: VDD_3V3D -> /Module_A3/HS_DIFF_0_N
- J3 pad 27: GND -> /Module_A3/HS_DIFF_1_P
- J3 pad 28: VDD_1V8D -> /Module_A3/HS_DIFF_0_P
- J3 pad 29: Net-(J3-Pad29) -> /Module_A3/HS_DIFF_3_N
- J3 pad 3: /Module_A3/MOD_SPI_MISO -> VDD_5V5A
- J3 pad 30: /Module_A3/LS_VREF -> /Module_A3/HS_DIFF_2_N
- J3 pad 31: GND -> /Module_A3/HS_DIFF_3_P
- J3 pad 32: /Module_A3/HS_VREF -> /Module_A3/HS_DIFF_2_P
- J3 pad 33: Net-(J3-Pad33) -> GND
- J3 pad 35: /Module_A3/HS_DIFF_CLK1_N -> /Module_A3/HS_DIFF_5_N
- J3 pad 36: /Module_A3/HS_DIFF_CLK0_N -> /Module_A3/HS_DIFF_4_N
- J3 pad 37: /Module_A3/HS_DIFF_CLK1_P -> /Module_A3/HS_DIFF_5_P
- J3 pad 38: /Module_A3/HS_DIFF_CLK0_P -> /Module_A3/HS_DIFF_4_P
- J3 pad 39: GND -> /Module_A3/HS_DIFF_7_N
- J3 pad 40: GND -> /Module_A3/HS_DIFF_6_N
- J3 pad 41: /Module_A3/HS_DIFF_15_N -> /Module_A3/HS_DIFF_7_P
- J3 pad 42: /Module_A3/HS_DIFF_7_N -> /Module_A3/HS_DIFF_6_P
- J3 pad 43: /Module_A3/HS_DIFF_15_P -> /Module_A3/HS_DIFF_9_N
- J3 pad 44: /Module_A3/HS_DIFF_7_P -> /Module_A3/HS_DIFF_8_N
- J3 pad 45: /Module_A3/HS_DIFF_14_N -> /Module_A3/HS_DIFF_9_P
- J3 pad 46: /Module_A3/HS_DIFF_6_N -> /Module_A3/HS_DIFF_8_P
- J3 pad 47: /Module_A3/HS_DIFF_14_P -> GND
- J3 pad 48: /Module_A3/HS_DIFF_6_P -> GND
- J3 pad 49: GND -> /Module_A3/HS_DIFF_11_N
- J3 pad 5: /Module_A3/MOD_SPI_SCK -> VDD_3V3D
- J3 pad 50: GND -> /Module_A3/HS_DIFF_10_N
- J3 pad 51: /Module_A3/HS_DIFF_13_N -> /Module_A3/HS_DIFF_11_P
- J3 pad 52: /Module_A3/HS_DIFF_5_N -> /Module_A3/HS_DIFF_10_P
- J3 pad 53: /Module_A3/HS_DIFF_13_P -> /Module_A3/HS_DIFF_13_N
- J3 pad 54: /Module_A3/HS_DIFF_5_P -> /Module_A3/HS_DIFF_12_N
- J3 pad 55: /Module_A3/HS_DIFF_12_N -> /Module_A3/HS_DIFF_13_P
- J3 pad 56: /Module_A3/HS_DIFF_4_N -> /Module_A3/HS_DIFF_12_P
- J3 pad 57: /Module_A3/HS_DIFF_12_P -> /Module_A3/HS_DIFF_15_N
- J3 pad 58: /Module_A3/HS_DIFF_4_P -> /Module_A3/HS_DIFF_14_N
- J3 pad 59: GND -> /Module_A3/HS_DIFF_15_P
- J3 pad 60: GND -> /Module_A3/HS_DIFF_14_P
- J3 pad 61: /Module_A3/HS_DIFF_11_N -> GND
- J3 pad 62: /Module_A3/HS_DIFF_3_N -> GND
- J3 pad 63: /Module_A3/HS_DIFF_11_P -> /Module_A3/LS_GPIO4
- J3 pad 64: /Module_A3/HS_DIFF_3_P -> /Module_A3/LS_VREF
- J3 pad 65: /Module_A3/HS_DIFF_10_N -> /Module_A3/LS_GPIO5
- J3 pad 66: /Module_A3/HS_DIFF_2_N -> /Module_A3/MOD_SPI_SCK
- J3 pad 67: /Module_A3/HS_DIFF_10_P -> /Module_A3/LS_GPIO6
- J3 pad 68: /Module_A3/HS_DIFF_2_P -> /Module_A3/MOD_SPI_MISO
- J3 pad 69: GND -> /Module_A3/I2C_A2
- J3 pad 7: /Module_A3/LS_GPIO0 -> VDD_3V3D
- J3 pad 70: GND -> /Module_A3/MOD_SPI_MOSI
- J3 pad 71: /Module_A3/HS_DIFF_9_N -> /Module_A3/I2C_A1
- J3 pad 72: /Module_A3/HS_DIFF_1_N -> /Module_A3/LS_GPIO0
- J3 pad 73: /Module_A3/HS_DIFF_9_P -> /Module_A3/I2C_A0
- J3 pad 74: /Module_A3/HS_DIFF_1_P -> /Module_A3/LS_GPIO1
- J3 pad 75: /Module_A3/HS_DIFF_8_N -> /Module_A3/I2C_SDA
- J3 pad 76: /Module_A3/HS_DIFF_0_N -> /Module_A3/LS_GPIO2
- J3 pad 77: /Module_A3/HS_DIFF_8_P -> /Module_A3/I2C_SCL
- J3 pad 78: /Module_A3/HS_DIFF_0_P -> /Module_A3/LS_GPIO3
- J3 pad 8: VDD_SYSTEM -> VDD_1V8D
- J3 pad 9: /Module_A3/LS_GPIO1 -> GND
- J4 pad 1: /Module_A4/MOD_SPI_MOSI -> VDD_5V5A
- J4 pad 10: VDD_SYSTEM -> unconnected-(J4-Pad10)
- J4 pad 11: /Module_A4/LS_GPIO2 -> Net-(J4-Pad11)
- J4 pad 12: GND -> unconnected-(J4-Pad12)
- J4 pad 13: /Module_A4/LS_GPIO3 -> GND
- J4 pad 14: VDD_5V5A -> /Module_A4/HS_VREF
- J4 pad 15: /Module_A4/LS_GPIO4 -> Net-(J4-Pad15)
- J4 pad 16: VDD_5V5A -> unconnected-(J4-Pad16)
- J4 pad 17: /Module_A4/LS_GPIO5 -> GND
- J4 pad 18: VDD_5V5A -> GND
- J4 pad 19: /Module_A4/LS_GPIO6 -> /Module_A4/HS_DIFF_CLK0_P
- J4 pad 20: GND -> /Module_A4/HS_DIFF_CLK1_P
- J4 pad 21: /Module_A4/LS_GPIO7 -> /Module_A4/HS_DIFF_CLK0_N
- J4 pad 22: GND -> /Module_A4/HS_DIFF_CLK1_N
- J4 pad 23: /Module_A4/LS_GPIO8 -> GND
- J4 pad 24: VDD_3V3D -> GND
- J4 pad 25: /Module_A4/LS_GPIO9 -> /Module_A4/HS_DIFF_1_N
- J4 pad 26: VDD_3V3D -> /Module_A4/HS_DIFF_0_N
- J4 pad 27: GND -> /Module_A4/HS_DIFF_1_P
- J4 pad 28: VDD_1V8D -> /Module_A4/HS_DIFF_0_P
- J4 pad 29: Net-(J4-Pad29) -> /Module_A4/HS_DIFF_3_N
- J4 pad 3: /Module_A4/MOD_SPI_MISO -> VDD_5V5A
- J4 pad 30: /Module_A4/LS_VREF -> /Module_A4/HS_DIFF_2_N
- J4 pad 31: GND -> /Module_A4/HS_DIFF_3_P
- J4 pad 32: /Module_A4/HS_VREF -> /Module_A4/HS_DIFF_2_P
- J4 pad 33: Net-(J4-Pad33) -> GND
- J4 pad 35: /Module_A4/HS_DIFF_CLK1_N -> /Module_A4/HS_DIFF_5_N
- J4 pad 36: /Module_A4/HS_DIFF_CLK0_N -> /Module_A4/HS_DIFF_4_N
- J4 pad 37: /Module_A4/HS_DIFF_CLK1_P -> /Module_A4/HS_DIFF_5_P
- J4 pad 38: /Module_A4/HS_DIFF_CLK0_P -> /Module_A4/HS_DIFF_4_P
- J4 pad 39: GND -> /Module_A4/HS_DIFF_7_N
- J4 pad 40: GND -> /Module_A4/HS_DIFF_6_N
- J4 pad 41: /Module_A4/HS_DIFF_15_N -> /Module_A4/HS_DIFF_7_P
- J4 pad 42: /Module_A4/HS_DIFF_7_N -> /Module_A4/HS_DIFF_6_P
- J4 pad 43: /Module_A4/HS_DIFF_15_P -> /Module_A4/HS_DIFF_9_N
- J4 pad 44: /Module_A4/HS_DIFF_7_P -> /Module_A4/HS_DIFF_8_N
- J4 pad 45: /Module_A4/HS_DIFF_14_N -> /Module_A4/HS_DIFF_9_P
- J4 pad 46: /Module_A4/HS_DIFF_6_N -> /Module_A4/HS_DIFF_8_P
- J4 pad 47: /Module_A4/HS_DIFF_14_P -> GND
- J4 pad 48: /Module_A4/HS_DIFF_6_P -> GND
- J4 pad 49: GND -> /Module_A4/HS_DIFF_11_N
- J4 pad 5: /Module_A4/MOD_SPI_SCK -> VDD_3V3D
- J4 pad 50: GND -> /Module_A4/HS_DIFF_10_N
- J4 pad 51: /Module_A4/HS_DIFF_13_N -> /Module_A4/HS_DIFF_11_P
- J4 pad 52: /Module_A4/HS_DIFF_5_N -> /Module_A4/HS_DIFF_10_P
- J4 pad 53: /Module_A4/HS_DIFF_13_P -> /Module_A4/HS_DIFF_13_N
- J4 pad 54: /Module_A4/HS_DIFF_5_P -> /Module_A4/HS_DIFF_12_N
- J4 pad 55: /Module_A4/HS_DIFF_12_N -> /Module_A4/HS_DIFF_13_P
- J4 pad 56: /Module_A4/HS_DIFF_4_N -> /Module_A4/HS_DIFF_12_P
- J4 pad 57: /Module_A4/HS_DIFF_12_P -> /Module_A4/HS_DIFF_15_N
- J4 pad 58: /Module_A4/HS_DIFF_4_P -> /Module_A4/HS_DIFF_14_N
- J4 pad 59: GND -> /Module_A4/HS_DIFF_15_P
- J4 pad 60: GND -> /Module_A4/HS_DIFF_14_P
- J4 pad 61: /Module_A4/HS_DIFF_11_N -> GND
- J4 pad 62: /Module_A4/HS_DIFF_3_N -> GND
- J4 pad 63: /Module_A4/HS_DIFF_11_P -> /Module_A4/LS_GPIO4
- J4 pad 64: /Module_A4/HS_DIFF_3_P -> /Module_A4/LS_VREF
- J4 pad 65: /Module_A4/HS_DIFF_10_N -> /Module_A4/LS_GPIO5
- J4 pad 66: /Module_A4/HS_DIFF_2_N -> /Module_A4/MOD_SPI_SCK
- J4 pad 67: /Module_A4/HS_DIFF_10_P -> /Module_A4/LS_GPIO6
- J4 pad 68: /Module_A4/HS_DIFF_2_P -> /Module_A4/MOD_SPI_MISO
- J4 pad 69: GND -> /Module_A4/I2C_A2
- J4 pad 7: /Module_A4/LS_GPIO0 -> VDD_3V3D
- J4 pad 70: GND -> /Module_A4/MOD_SPI_MOSI
- J4 pad 71: /Module_A4/HS_DIFF_9_N -> /Module_A4/I2C_A1
- J4 pad 72: /Module_A4/HS_DIFF_1_N -> /Module_A4/LS_GPIO0
- J4 pad 73: /Module_A4/HS_DIFF_9_P -> /Module_A4/I2C_A0
- J4 pad 74: /Module_A4/HS_DIFF_1_P -> /Module_A4/LS_GPIO1
- J4 pad 75: /Module_A4/HS_DIFF_8_N -> /Module_A4/I2C_SDA
- J4 pad 76: /Module_A4/HS_DIFF_0_N -> /Module_A4/LS_GPIO2
- J4 pad 77: /Module_A4/HS_DIFF_8_P -> /Module_A4/I2C_SCL
- J4 pad 78: /Module_A4/HS_DIFF_0_P -> /Module_A4/LS_GPIO3
- J4 pad 8: VDD_SYSTEM -> VDD_1V8D
- J4 pad 9: /Module_A4/LS_GPIO1 -> GND
- R1 pad 1: Net-(J1-Pad29) -> Net-(J1-Pad11)
- R2 pad 1: Net-(J2-Pad29) -> Net-(J2-Pad11)
- R3 pad 1: Net-(J2-Pad33) -> Net-(J2-Pad15)
- R4 pad 1: Net-(J3-Pad29) -> Net-(J3-Pad11)
- R5 pad 1: Net-(J1-Pad33) -> Net-(J1-Pad15)
- R6 pad 1: Net-(J3-Pad33) -> Net-(J3-Pad15)
- R7 pad 1: Net-(J4-Pad29) -> Net-(J4-Pad11)
- R8 pad 1: Net-(J4-Pad33) -> Net-(J4-Pad15)
- U1 pad A11: unconnected-(U1D-PS_MIO28_501-PadA11) -> /Zynq_PSMIO/MIO_RGMII_TX_CLK
- U1 pad A12: unconnected-(U1D-PS_MIO30_501-PadA12) -> /Zynq_PSMIO/MIO_RGMII_TX1
- U1 pad A13: Net-(U1F-VCCO_MIO1_501-PadA13) -> VCC_MIO
- U1 pad A14: unconnected-(U1D-PS_MIO36_501-PadA14) -> /Zynq_PSMIO/MIO_RGMII_RX1
- U1 pad A15: unconnected-(U1D-PS_MIO20_501-PadA15) -> /Zynq_PSMIO/MIO_SD_D2
- U1 pad A16: unconnected-(U1D-PS_MIO18_501-PadA16) -> /Zynq_PSMIO/MIO_SD_D0
- U1 pad A19: unconnected-(U1D-PS_MIO6_500-PadA19) -> /Zynq_PSMIO/MIO_QSPI_SCLK
- U1 pad A20: unconnected-(U1D-PS_MIO5_500-PadA20) -> /Zynq_PSMIO/MIO_QSPI_IO3
- U1 pad A21: unconnected-(U1D-PS_MIO2_500-PadA21) -> /Zynq_PSMIO/MIO_QSPI_IO0
- U1 pad A22: unconnected-(U1D-PS_MIO1_500-PadA22) -> /Zynq_PSMIO/MIO_QSPI_CS
- U1 pad AA3: Net-(U1A-MGTPTXP0_112) -> Net-(U1J-MGTPTXP0_112)
- U1 pad AA5: Net-(U1A-MGTPTXP2_112) -> Net-(U1J-MGTPTXP2_112)
- U1 pad AA7: Net-(U1A-MGTPRXP0_112) -> Net-(U1J-MGTPRXP0_112)
- U1 pad AA9: Net-(U1A-MGTPRXP2_112) -> Net-(U1J-MGTPRXP2_112)
- U1 pad AB3: Net-(U1A-MGTPTXN0_112) -> Net-(U1J-MGTPTXN0_112)
- U1 pad AB5: Net-(U1A-MGTPTXN2_112) -> Net-(U1J-MGTPTXN2_112)
- U1 pad AB7: Net-(U1A-MGTPRXN0_112) -> Net-(U1J-MGTPRXN0_112)
- U1 pad AB9: Net-(U1A-MGTPRXN2_112) -> Net-(U1J-MGTPRXN2_112)
- U1 pad B10: Net-(U1F-VCCO_MIO1_501-PadA13) -> VCC_MIO
- U1 pad B11: unconnected-(U1D-PS_MIO34_501-PadB11) -> /Zynq_PSMIO/MIO_RGMII_RX_CLK
- U1 pad B12: unconnected-(U1D-PS_MIO43_501-PadB12) -> /Zynq_PSMIO/MIO_ULPI_NXT
- U1 pad B13: unconnected-(U1D-PS_MIO47_501-PadB13) -> /Zynq_PSMIO/MIO_ULPI_D3
- U1 pad B14: unconnected-(U1D-PS_MIO45_501-PadB14) -> /Zynq_PSMIO/MIO_ULPI_D1
- U1 pad B20: Net-(U1F-VCCO_MIO0_500-PadB20) -> VCC_MIO
- U1 pad B9: unconnected-(U1D-PS_MIO37_501-PadB9) -> /Zynq_PSMIO/MIO_RGMII_RX2
- U1 pad C10: unconnected-(U1D-PS_MIO39_501-PadC10) -> /Zynq_PSMIO/MIO_RGMII_RX_CTL
- U1 pad C13: unconnected-(U1D-PS_MIO51_501-PadC13) -> /Zynq_PSMIO/MIO_ULPI_D7
- U1 pad C15: unconnected-(U1D-PS_MIO41_501-PadC15) -> /Zynq_PSMIO/MIO_ULPI_DIR
- U1 pad C16: unconnected-(U1D-PS_MIO32_501-PadC16) -> /Zynq_PSMIO/MIO_RGMII_TX3
- U1 pad C17: Net-(U1F-VCCO_MIO0_500-PadB20) -> VCC_MIO
- U1 pad C9: unconnected-(U1D-PS_MIO49_501-PadC9) -> /Zynq_PSMIO/MIO_ULPI_D5
- U1 pad D10: unconnected-(U1D-PS_MIO50_501-PadD10) -> /Zynq_PSMIO/MIO_ULPI_D6
- U1 pad D11: unconnected-(U1D-PS_MIO46_501-PadD11) -> /Zynq_PSMIO/MIO_ULPI_D2
- U1 pad D12: unconnected-(U1D-PS_MIO48_501-PadD12) -> /Zynq_PSMIO/MIO_ULPI_CLK
- U1 pad D14: Net-(U1F-VCCO_MIO1_501-PadA13) -> VCC_MIO
- U1 pad D15: unconnected-(U1D-PS_MIO42_501-PadD15) -> /Zynq_PSMIO/MIO_ULPI_STP
- U1 pad D17: unconnected-(U1D-PS_MIO16_501-PadD17) -> /Zynq_PSMIO/MIO_SD_CLK
- U1 pad E10: unconnected-(U1D-PS_MIO44_501-PadE10) -> /Zynq_PSMIO/MIO_ULPI_D0
- U1 pad E11: Net-(U1F-VCCO_MIO1_501-PadA13) -> VCC_MIO
- U1 pad E13: unconnected-(U1D-PS_MIO19_501-PadE13) -> /Zynq_PSMIO/MIO_SD_D1
- U1 pad E14: unconnected-(U1D-PS_MIO17_501-PadE14) -> /Zynq_PSMIO/MIO_SD_CMD
- U1 pad E15: unconnected-(U1D-PS_MIO29_501-PadE15) -> /Zynq_PSMIO/MIO_RGMII_TX0
- U1 pad E18: unconnected-(U1D-PS_MIO8_500-PadE18) -> /Zynq_PSMIO/MIO_QSPI_FB
- U1 pad E19: unconnected-(U1D-PS_MIO4_500-PadE19) -> /Zynq_PSMIO/MIO_QSPI_IO2
- U1 pad E9: unconnected-(U1D-PS_MIO40_501-PadE9) -> /Zynq_PSMIO/MIO_ULPI_D4
- U1 pad F10: unconnected-(U1D-PS_MIO38_501-PadF10) -> /Zynq_PSMIO/MIO_RGMII_RX3
- U1 pad F12: unconnected-(U1D-PS_MIO21_501-PadF12) -> /Zynq_PSMIO/MIO_SD_D3
- U1 pad F14: unconnected-(U1D-PS_MIO31_501-PadF14) -> /Zynq_PSMIO/MIO_RGMII_TX2
- U1 pad F17: unconnected-(U1D-PS_MIO3_500-PadF17) -> /Zynq_PSMIO/MIO_QSPI_IO1
- U1 pad F9: unconnected-(U1D-PS_MIO35_501-PadF9) -> /Zynq_PSMIO/MIO_RGMII_RX0
- U1 pad G11: unconnected-(U1D-PS_MIO33_501-PadG11) -> /Zynq_PSMIO/MIO_RGMII_TX_CTL
- U1 pad G15: /ZynqPower/PS_CORE -> /ZynqPower/1V_RAIL_A
- U1 pad H12: /ZynqPower/VCCBRAM -> /ZynqPower/1V_RAIL_B
- U1 pad H14: /ZynqPower/PS_CORE -> /ZynqPower/1V_RAIL_A
- U1 pad H8: unconnected-(U1A-IO_0_34-PadH8) -> (no net)
- U1 pad J1: unconnected-(U1B-IO_L8N_T1_34-PadJ1) -> (no net)
- U1 pad J11: /ZynqPower/VCCINT -> /ZynqPower/1V_RAIL_B
- U1 pad J13: /ZynqPower/VCCBRAM -> /ZynqPower/1V_RAIL_B
- U1 pad J15: /ZynqPower/PS_CORE -> /ZynqPower/1V_RAIL_A
- U1 pad J2: unconnected-(U1B-IO_L8P_T1_34-PadJ2) -> (no net)
- U1 pad J3: unconnected-(U1B-IO_L9P_T1_DQS_34-PadJ3) -> (no net)
- U1 pad J5: unconnected-(U1B-IO_L7P_T1_34-PadJ5) -> (no net)
- U1 pad J6: unconnected-(U1B-IO_L2N_T0_34-PadJ6) -> (no net)
- U1 pad J7: unconnected-(U1B-IO_L2P_T0_34-PadJ7) -> (no net)
- U1 pad J8: unconnected-(U1B-IO_L1P_T0_34-PadJ8) -> (no net)
- U1 pad J9: /ZynqPower/VCCINT -> /ZynqPower/1V_RAIL_B
- U1 pad K10: /ZynqPower/VCCINT -> /ZynqPower/1V_RAIL_B
- U1 pad K14: /ZynqPower/VCCPAUX -> /ZynqPower/1V8_RAIL_A
- U1 pad K2: unconnected-(U1B-IO_L9N_T1_DQS_34-PadK2) -> (no net)
- U1 pad K3: unconnected-(U1B-IO_L11N_T1_SRCC_34-PadK3) -> (no net)
- U1 pad K4: unconnected-(U1B-IO_L11P_T1_SRCC_34-PadK4) -> (no net)
- U1 pad K5: unconnected-(U1B-IO_L7N_T1_34-PadK5) -> (no net)
- U1 pad K7: unconnected-(U1B-IO_L3P_T0_DQS_PUDC_B_34-PadK7) -> (no net)
- U1 pad K8: unconnected-(U1B-IO_L1N_T0_34-PadK8) -> (no net)
- U1 pad L1: unconnected-(U1B-IO_L10N_T1_34-PadL1) -> (no net)
- U1 pad L13: /ZynqPower/VCCPAUX -> /ZynqPower/1V8_RAIL_A
- U1 pad L15: /ZynqPower/PS_CORE -> /ZynqPower/1V_RAIL_A
- U1 pad L2: unconnected-(U1B-IO_L10P_T1_34-PadL2) -> (no net)
- U1 pad L4: unconnected-(U1B-IO_L12N_T1_MRCC_34-PadL4) -> (no net)
- U1 pad L5: unconnected-(U1B-IO_L12P_T1_MRCC_34-PadL5) -> (no net)
- U1 pad L6: unconnected-(U1B-IO_L4P_T0_34-PadL6) -> (no net)
- U1 pad L7: unconnected-(U1B-IO_L3N_T0_DQS_34-PadL7) -> (no net)
- U1 pad L9: /ZynqPower/VCCINT -> /ZynqPower/1V_RAIL_B
- U1 pad M1: unconnected-(U1B-IO_L15N_T2_DQS_34-PadM1) -> (no net)
- U1 pad M10: /ZynqPower/VCCINT -> /ZynqPower/1V_RAIL_B
- U1 pad M14: /ZynqPower/VCCPAUX -> /ZynqPower/1V8_RAIL_A
- U1 pad M2: unconnected-(U1B-IO_L15P_T2_DQS_34-PadM2) -> (no net)
- U1 pad M3: unconnected-(U1A-IO_L22N_T3_34-PadM3) -> (no net)
- U1 pad M4: unconnected-(U1A-IO_L22P_T3_34-PadM4) -> (no net)
- U1 pad M6: unconnected-(U1B-IO_L4N_T0_34-PadM6) -> (no net)
- U1 pad M7: unconnected-(U1E-IO_L6N_T0_VREF_34-PadM7) -> (no net)
- U1 pad M8: unconnected-(U1B-IO_L6P_T0_34-PadM8) -> (no net)
- U1 pad N1: unconnected-(U1A-IO_L16P_T2_34-PadN1) -> (no net)
- U1 pad N13: /ZynqPower/VCCAUX -> VCC_MIO
- U1 pad N15: /ZynqPower/PS_CORE -> /ZynqPower/1V_RAIL_A
- U1 pad N3: unconnected-(U1A-IO_L21N_T3_DQS_34-PadN3) -> (no net)
- U1 pad N4: unconnected-(U1A-IO_L21P_T3_DQS_34-PadN4) -> (no net)
- U1 pad N5: unconnected-(U1E-IO_L19N_T3_VREF_34-PadN5) -> (no net)
- U1 pad N6: unconnected-(U1A-IO_L19P_T3_34-PadN6) -> (no net)
- U1 pad N8: unconnected-(U1B-IO_L5P_T0_34-PadN8) -> (no net)
- U1 pad N9: /ZynqPower/VCCINT -> /ZynqPower/1V_RAIL_B
- U1 pad P1: unconnected-(U1A-IO_L16N_T2_34-PadP1) -> (no net)
- U1 pad P10: /ZynqPower/VCCINT -> /ZynqPower/1V_RAIL_B
- U1 pad P12: /ZynqPower/VCCAUX -> VCC_MIO
- U1 pad P14: /ZynqPower/VCCPAUX -> /ZynqPower/1V8_RAIL_A
- U1 pad P2: unconnected-(U1A-IO_L18N_T2_34-PadP2) -> (no net)
- U1 pad P3: unconnected-(U1A-IO_L18P_T2_34-PadP3) -> (no net)
- U1 pad P5: unconnected-(U1A-IO_L20N_T3_34-PadP5) -> (no net)
- U1 pad P6: unconnected-(U1A-IO_L20P_T3_34-PadP6) -> (no net)
- U1 pad P7: unconnected-(U1A-IO_L24P_T3_34-PadP7) -> (no net)
- U1 pad P8: unconnected-(U1B-IO_L5N_T0_34-PadP8) -> (no net)
- U1 pad R13: /ZynqPower/VCCAUX -> VCC_MIO
- U1 pad R15: /ZynqPower/PS_CORE -> /ZynqPower/1V_RAIL_A
- U1 pad R2: unconnected-(U1A-IO_L17N_T2_34-PadR2) -> (no net)
- U1 pad R3: unconnected-(U1A-IO_L17P_T2_34-PadR3) -> (no net)
- U1 pad R4: unconnected-(U1A-IO_L23N_T3_34-PadR4) -> (no net)
- U1 pad R5: unconnected-(U1A-IO_L23P_T3_34-PadR5) -> (no net)
- U1 pad R7: unconnected-(U1A-IO_L24N_T3_34-PadR7) -> (no net)
- U1 pad R8: unconnected-(U1A-IO_25_34-PadR8) -> (no net)
- U1 pad R9: /ZynqPower/VCCINT -> /ZynqPower/1V_RAIL_B
- U1 pad T1: unconnected-(U1B-IO_L13N_T2_MRCC_34-PadT1) -> (no net)
- U1 pad T12: /ZynqPower/VCCAUX -> VCC_MIO
- U1 pad T2: unconnected-(U1B-IO_L13P_T2_MRCC_34-PadT2) -> (no net)
- U1 pad U1: unconnected-(U1B-IO_L14N_T2_SRCC_34-PadU1) -> (no net)
- U1 pad U2: unconnected-(U1B-IO_L14P_T2_SRCC_34-PadU2) -> (no net)
- U1 pad U5: Net-(U1A-MGTREFCLK1P_112) -> Net-(U1J-MGTREFCLK1P_112)
- U1 pad U9: Net-(U1A-MGTREFCLK0P_112) -> Net-(U1J-MGTREFCLK0P_112)
- U1 pad V5: Net-(U1A-MGTREFCLK1N_112) -> Net-(U1J-MGTREFCLK1N_112)
- U1 pad V9: Net-(U1A-MGTREFCLK0N_112) -> Net-(U1J-MGTREFCLK0N_112)
- U1 pad W2: Net-(U1A-MGTPTXP3_112) -> Net-(U1J-MGTPTXP3_112)
- U1 pad W4: Net-(U1A-MGTPTXP1_112) -> Net-(U1J-MGTPTXP1_112)
- U1 pad W6: Net-(U1A-MGTPRXP3_112) -> Net-(U1J-MGTPRXP3_112)
- U1 pad W8: Net-(U1A-MGTPRXP1_112) -> Net-(U1J-MGTPRXP1_112)
- U1 pad Y2: Net-(U1A-MGTPTXN3_112) -> Net-(U1J-MGTPTXN3_112)
- U1 pad Y4: Net-(U1A-MGTPTXN1_112) -> Net-(U1J-MGTPTXN1_112)
- U1 pad Y6: Net-(U1A-MGTPRXN3_112) -> Net-(U1J-MGTPRXN3_112)
- U5 pad A1: Net-(U5-OUT) -> VCC_MIO
Routing:
- net (no net): track 0.00 -> 78.2 mm, vias 0 -> 10
- net VCC_MIO: track 0.00 -> 54.9 mm, vias 0 -> 10
- net /GT_RX3_N: track 0.00 -> 41.0 mm, vias 0 -> 1
- net /GT_RX0_N: track 0.00 -> 40.4 mm, vias 0 -> 1
- net unconnected-(U1K-IO_L20P_T3_13-PadU19): track 0.00 -> 39.8 mm, vias 0 -> 2
- net unconnected-(U1K-IO_L23N_T3_13-PadW16): track 0.00 -> 39.6 mm, vias 0 -> 2
- net unconnected-(U1K-IO_L24P_T3_13-PadW17): track 0.00 -> 39.6 mm, vias 0 -> 2
- net /GTP_REF_CLK1_P: track 0.00 -> 38.6 mm, vias 0 -> 2
- net unconnected-(U1K-IO_L2N_T0_13-PadW15): track 0.00 -> 38.1 mm, vias 0 -> 2
- net /GTP_REF_CLK1_N: track 0.00 -> 37.9 mm, vias 0 -> 2
- net /GT_RX3_P: track 0.00 -> 37.5 mm, vias 0 -> 1
- net /ZynqPower/1V_RAIL_A: track 0.00 -> 36.9 mm, vias 0 -> 6
- net /GT_RX0_P: track 0.00 -> 36.9 mm, vias 0 -> 1
- net /GT_TX3_N: track 0.00 -> 36.3 mm, vias 0 -> 2
- net unconnected-(U1B-IO_L5N_T0_AD9N_35-PadE5): track 4.92 -> 40.7 mm
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- added copper zone on In1.Cu, net /ZynqPower/1V8_RAIL_A
- added copper zone on In1.Cu, net /ZynqPower/1V_RAIL_A
- added copper zone on In1.Cu, net /ZynqPower/1V_RAIL_B
- added copper zone on In1.Cu, net VCC_MIO
- removed copper zone on In1.Cu, net /ZynqPower/PS_CORE
- removed copper zone on In1.Cu, net /ZynqPower/VCCAUX
- removed copper zone on In1.Cu, net /ZynqPower/VCCINT
- removed copper zone on In1.Cu, net /ZynqPower/VCCPAUX

Commit message: V0.2
Connections:
- net /Module_A1/HS_DIFF_7_N renamed /A1_HS_7_N
- net /Module_A1/HS_DIFF_7_P renamed /A1_HS_7_P
- net /Module_A1/HS_DIFF_CLK1_N renamed /A1_HS1_CLK_N
- net /Module_A1/HS_DIFF_CLK1_P renamed /A1_HS1_CLK_P
- net /Module_A2/HS_DIFF_0_N renamed /A2_HS_0_N
- net /Module_A2/HS_DIFF_0_P renamed /A2_HS_0_P
- net /Module_A2/HS_DIFF_10_N renamed /A2_HS_10_N
- net /Module_A2/HS_DIFF_10_P renamed /A2_HS_10_P
- net /Module_A2/HS_DIFF_11_N renamed /A2_HS_11_N
- net /Module_A2/HS_DIFF_11_P renamed /A2_HS_11_P
- net /Module_A2/HS_DIFF_12_N renamed /A2_HS_12_N
- net /Module_A2/HS_DIFF_12_P renamed /A2_HS_12_P
- net /Module_A2/HS_DIFF_13_N renamed /A2_HS_13_N
- net /Module_A2/HS_DIFF_13_P renamed /A2_HS_13_P
- net /Module_A2/HS_DIFF_14_N renamed /A2_HS_14_N
- net /Module_A2/HS_DIFF_14_P renamed /A2_HS_14_P
- net /Module_A2/HS_DIFF_15_N renamed /A2_HS_15_N
- net /Module_A2/HS_DIFF_15_P renamed /A2_HS_15_P
- net /Module_A2/HS_DIFF_1_N renamed /A2_HS_1_N
- net /Module_A2/HS_DIFF_1_P renamed /A2_HS_1_P
- net /Module_A2/HS_DIFF_2_N renamed /A2_HS_2_N
- net /Module_A2/HS_DIFF_2_P renamed /A2_HS_2_P
- net /Module_A2/HS_DIFF_3_N renamed /A2_HS_3_N
- net /Module_A2/HS_DIFF_3_P renamed /A2_HS_3_P
- net /Module_A2/HS_DIFF_4_N renamed /A2_HS_4_N
- net /Module_A2/HS_DIFF_4_P renamed /A2_HS_4_P
- net /Module_A2/HS_DIFF_5_N renamed /A2_HS_5_N
- net /Module_A2/HS_DIFF_5_P renamed /A2_HS_5_P
- net /Module_A2/HS_DIFF_6_N renamed /A2_HS_6_N
- net /Module_A2/HS_DIFF_6_P renamed /A2_HS_6_P
- net /Module_A2/HS_DIFF_7_N renamed /A2_HS_7_N
- net /Module_A2/HS_DIFF_7_P renamed /A2_HS_7_P
- net /Module_A2/HS_DIFF_8_N renamed /A2_HS_8_N
- net /Module_A2/HS_DIFF_8_P renamed /A2_HS_8_P
- net /Module_A2/HS_DIFF_9_N renamed /A2_HS_9_N
- net /Module_A2/HS_DIFF_9_P renamed /A2_HS_9_P
- net /Module_A2/HS_DIFF_CLK0_N renamed /A2_HS0_CLK_N
- net /Module_A2/HS_DIFF_CLK0_P renamed /A2_HS0_CLK_P
- net /Module_A2/HS_DIFF_CLK1_N renamed /A2_HS1_CLK_N
- net /Module_A2/HS_DIFF_CLK1_P renamed /A2_HS1_CLK_P
- J1 pad 35: /Module_A1/HS_DIFF_5_N -> /A1_HS_5_N
- J1 pad 36: /Module_A1/HS_DIFF_4_N -> /A1_HS_4_N
- J1 pad 37: /Module_A1/HS_DIFF_5_P -> /A1_HS_5_P
- J1 pad 38: /Module_A1/HS_DIFF_4_P -> /A1_HS_4_P
- J1 pad 40: /Module_A1/HS_DIFF_6_N -> /A1_HS_6_N
- J1 pad 42: /Module_A1/HS_DIFF_6_P -> /A1_HS_6_P
- J1 pad 43: /Module_A1/HS_DIFF_9_N -> /A1_HS_9_N
- J1 pad 44: /Module_A1/HS_DIFF_8_N -> /A1_HS_8_N
- J1 pad 45: /Module_A1/HS_DIFF_9_P -> /A1_HS_9_P
- J1 pad 46: /Module_A1/HS_DIFF_8_P -> /A1_HS_8_P
- J1 pad 49: /Module_A1/HS_DIFF_11_N -> /A1_HS_11_N
- J1 pad 50: /Module_A1/HS_DIFF_10_N -> /A1_HS_10_N
- J1 pad 51: /Module_A1/HS_DIFF_11_P -> /A1_HS_11_P
- J1 pad 52: /Module_A1/HS_DIFF_10_P -> /A1_HS_10_P
- J1 pad 53: /Module_A1/HS_DIFF_13_N -> /A1_HS_13_N
- J1 pad 54: /Module_A1/HS_DIFF_12_N -> /A1_HS_12_N
- J1 pad 55: /Module_A1/HS_DIFF_13_P -> /A1_HS_13_P
- J1 pad 56: /Module_A1/HS_DIFF_12_P -> /A1_HS_12_P
- J1 pad 57: /Module_A1/HS_DIFF_15_N -> /A1_HS_15_N
- J1 pad 58: /Module_A1/HS_DIFF_14_N -> /A1_HS_14_N
- J1 pad 59: /Module_A1/HS_DIFF_15_P -> /A1_HS_15_P
- J1 pad 60: /Module_A1/HS_DIFF_14_P -> /A1_HS_14_P
- U1 pad AA11: unconnected-(U1K-IO_L7P_T1_13-PadAA11) -> /A1_HS_4_P
- U1 pad AA12: unconnected-(U1K-IO_L8P_T1_13-PadAA12) -> /A1_HS_6_P
- U1 pad AA14: unconnected-(U1K-IO_L11P_T1_SRCC_13-PadAA14) -> /A1_HS_11_P
- U1 pad AA15: unconnected-(U1K-IO_L11N_T1_SRCC_13-PadAA15) -> /A1_HS_11_N
- U1 pad AA16: unconnected-(U1K-IO_L14P_T2_SRCC_13-PadAA16) -> /A1_HS_15_P
- U1 pad AA17: unconnected-(U1K-IO_L14N_T2_SRCC_13-PadAA17) -> /A1_HS_15_N
- U1 pad AB11: unconnected-(U1K-IO_L7N_T1_13-PadAB11) -> /A1_HS_4_N
- U1 pad AB12: unconnected-(U1K-IO_L8N_T1_13-PadAB12) -> /A1_HS_6_N
- U1 pad AB13: unconnected-(U1K-IO_L9P_T1_DQS_13-PadAB13) -> /A1_HS_8_P
- U1 pad AB14: unconnected-(U1K-IO_L9N_T1_DQS_13-PadAB14) -> /A1_HS_8_N
- U1 pad AB16: unconnected-(U1K-IO_L17P_T2_13-PadAB16) -> /A1_HS_13_P
- U1 pad AB17: unconnected-(U1K-IO_L17N_T2_13-PadAB17) -> /A1_HS_13_N
- U1 pad V11: unconnected-(U1K-IO_L4P_T0_13-PadV11) -> /A1_HS_5_P
- U1 pad V15: unconnected-(U1K-IO_L2P_T0_13-PadV15) -> /A1_HS_12_P
- U1 pad V16: unconnected-(U1K-IO_L23P_T3_13-PadV16) -> /A1_HS_14_P
- U1 pad W11: unconnected-(U1K-IO_L4N_T0_13-PadW11) -> /A1_HS_5_N
- U1 pad W12: unconnected-(U1K-IO_L3P_T0_DQS_13-PadW12) -> /A1_HS_9_P
- U1 pad W13: unconnected-(U1K-IO_L3N_T0_DQS_13-PadW13) -> /A1_HS_9_N
- U1 pad W15: unconnected-(U1K-IO_L2N_T0_13-PadW15) -> /A1_HS_12_N
- U1 pad W16: unconnected-(U1K-IO_L23N_T3_13-PadW16) -> /A1_HS_14_N
- U1 pad Y12: unconnected-(U1K-IO_L10P_T1_13-PadY12) -> /A1_HS_10_P
- U1 pad Y13: unconnected-(U1K-IO_L10N_T1_13-PadY13) -> /A1_HS_10_N
Routing:
- net unconnected-(U1K-IO_L23P_T3_13-PadV16): track 40.5 -> 0.00 mm, vias 2 -> 0
- net /A1_HS_14_P: track 0.00 -> 40.5 mm, vias 0 -> 2
- net /A1_HS_5_P: track 0.00 -> 40.1 mm, vias 0 -> 2
- net unconnected-(U1K-IO_L23N_T3_13-PadW16): track 39.6 -> 0.00 mm, vias 2 -> 0
- net /A1_HS_14_N: track 0.00 -> 39.6 mm, vias 0 -> 2
- net unconnected-(U1K-IO_L2P_T0_13-PadV15): track 39.3 -> 0.00 mm, vias 2 -> 0
- net /A1_HS_12_P: track 0.00 -> 39.3 mm, vias 0 -> 2
- net /A1_HS_5_N: track 0.00 -> 39.1 mm, vias 0 -> 2
- net unconnected-(U1K-IO_L2N_T0_13-PadW15): track 38.1 -> 0.00 mm, vias 2 -> 0
- net /A1_HS_12_N: track 0.00 -> 38.1 mm, vias 0 -> 2
- net /A1_HS_6_P: track 0.00 -> 37.1 mm
- net unconnected-(U1K-IO_L4P_T0_13-PadV11): track 37.0 -> 0.00 mm, vias 2 -> 0
- net unconnected-(U1K-IO_L14P_T2_SRCC_13-PadAA16): track 36.9 -> 0.00 mm, vias 2 -> 0
- net /A1_HS_15_P: track 0.00 -> 36.9 mm, vias 0 -> 2
- net unconnected-(U1K-IO_L3N_T0_DQS_13-PadW13): track 36.9 -> 0.00 mm, vias 2 -> 0
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