File: TRX055.01.01.PB.00.00/EthPair.kicad_sch (KiCad schematic)
At the start: 9 parts, among them T1 SM453229-231N7Y

Commit message: + add clocks + add PSU
Parts:
- C131, C132: JLCPCB Part # (none) -> C25744
- C133: footprint Capacitor_SMD:C_0402_1005Metric -> Capacitor_SMD:C_0201_0603Metric; JLCPCB Part # (none) -> C1581
- C134: JLCPCB Part # (none) -> C1588; Voltage 2000V -> 100V
- R55, R58: JLCPCB Part # (none) -> C25120
- R59: JLCPCB Part # (none) -> C25133
- T1: JLCPCB Part # (none) -> C6816858

Commit message: V0.1 - production, added brig-up comments
Parts:
- C131, C132: value 10P -> DNP
- R55, R58: value 49R9 -> DNP
Connections:
- no-connect marks 0 -> 1
Other:
- note added: "BUG: Cut connection between central tab and VDD."
- company: (none) -> Tronex s.r.o. / Tronex Group USA LLC
- title: (none) -> TRNX SDR Carrier board
Changed lines of the file:
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@@
 	(generator_version "9.0")
 	(paper "A4")
+	(title_block
+		(title "TRNX SDR Carrier board")
+		(date "2025-11-18")
+		(rev "0.1")
+		(company "Tronex s.r.o. / Tronex Group USA LLC")
+	)
+	(text "BUG:\nCut connection between central tab and VDD. "
+		(exclude_from_sim no)
+		(at 105.664 43.434 0)
+		(effects
+			(font
+				(size 1.27 1.27)
+				(color 255 0 21 1)
+			)
+		)
+	)
 	(junction
 		(at 133.35 78.74)
@@
 		(diameter 0)
 		(color 0 0 0 0)
+	)
+	(no_connect
+		(at 105.41 54.61)
 	)
 	(wire
@@
 			)
 		)
-		(property "Value" "10P"
+		(property "Value" "DNP"
 			(at 81.28 97.7899 0)
 			(effects
@@
 			)
 		)
-		(property "Value" "49R9"
+		(property "Value" "DNP"
 			(at 93.98 58.4199 90)
 			(effects
@@
 			)
 		)
-		(property "Value" "49R9"
+		(property "Value" "DNP"
 			(at 80.01 58.4199 90)
 			(effects
@@
 			)
 		)
-		(property "Value" "10P"
+		(property "Value" "DNP"
 			(at 95.25 97.7899 0)
 			(effects
