File: TRX055.01.01.PB.00.00/Main_Power.kicad_sch (KiCad schematic)
At the start: 12 parts, among them J21 GT-BTP30003-0720A-016A, J22 GT-BTP30003-0720A-016A

Commit message: V0.1 - production, added brig-up comments
Parts:
- added C279, C280: Cap, Capacitor_SMD:C_0402_1005Metric, symbol PPA-Pasive:Cap
- added C281, C287, C312: M1, Capacitor_SMD:C_0201_0603Metric, symbol PPA-Pasive:Cap
- added C282, C283, C284, C285, C286, C310, C311, C313, C314: 10M, Capacitor_SMD:C_0603_1608Metric, symbol PPA-Pasive:Cap
- added C369, C370, C371, C372, C373, C374, C375, C376, C377: 22M, Capacitor_SMD:C_0603_1608Metric, symbol PPA-Pasive:Cap
- added C391, C395, C396, C397: 100M, Capacitor_SMD:C_1206_3216Metric, symbol PPA-Pasive:Cap
- added D5: DSK34, Diode_SMD:D_SOD-123F, symbol Diode:CDBA340-HF
- added JP13, JP14: Jumper_2_Open, foot-ppa-passive:SolderJumper-2_P1.3mm_open_Pad1.0x1.5mm, symbol Jumper:Jumper_2_Open
- added L15, L16, L18: EXLA1V0402-4R7-R, foot-ppa-passive:EXLA1V04, symbol PPA-Pasive:Ind
- added R100, R99: 240, Resistor_SMD:R_0402_1005Metric, symbol PPA-Pasive:Res
- added R137, R139: 33, Resistor_SMD:R_0402_1005Metric, symbol PPA-Pasive:Res
- added R138, R140: NU, Resistor_SMD:R_0402_1005Metric, symbol PPA-Pasive:Res
- added R96, R97: 10K, Resistor_SMD:R_0402_1005Metric, symbol PPA-Pasive:Res
- added R98: 8K06, Resistor_SMD:R_0402_1005Metric, symbol PPA-Pasive:Res
- added U21, U30: AP63203WU, Package_TO_SOT_SMD:TSOT-23-6, symbol Regulator_Switching:AP63203WU
- added U27, U29: LM73100RPWR, ppa-active:VQFN-10_L2.0-W2.0-P0.45-TL, symbol ppa-ic-power:LM73100RPWR
Connections:
- net TPS5430DD_DCDC/FB_GND is gone; now on net GND: R3.2
- net TPS5430DD_DCDC1/FB_GND is gone; now on net GND: R94.2
- net GND: now also C279.2, C280.2, C282.2, C283.2, C284.2, C285.2, C286.2, C287.1, C310.2, C311.2, C313.2, C314.2, C369.2, C370.2, C371.2, C372.2, C373.2, C374.2, C375.2, C376.2, C377.2, C391.2, C395.2, C396.2, C397.2, R100.2, R138.2, R140.2, R96.2, R97.2, U21.4 (GND), U27.8 (GND), U29.2 (OVLO), U29.8 (GND), U30.4 (GND)
- net USB_PD_PWR: now also R98.2, U27.5 (IN)
- net at D2.2 (A), J21.2: now also D5.2 (A)
- net VDD_5V5A: now reaches JP9.2 (B)
- net VDD_5V5A: now also C310.1, C311.1, C396.1, C397.1, U21.3 (IN)
- net PWR_CORE: now reaches JP12.2 (B)
- net PWR_CORE: now also C391.1, C395.1
- net MAIN_PWR renamed VDD_MAIN_PWR
- net VDD_MAIN_PWR: now also C369.1, C370.1, C371.1, C372.1, C373.1, C374.1, C375.1, C376.1, C377.1, U27.6 (OUT), U29.5 (IN); no longer D1.1 (K)
- new net: C313.1, C314.1, JP14.1 (A), L18.2, R139.1
- new net: R139.2, R140.1, U21.1 (FB)
- new net: C282.1, C283.1, JP13.1 (A), L15.2, R137.1
- new net: R137.2, R138.1, U30.1 (FB)
- new net: C312.2, L18.1, U21.5 (SW)
- new net: R100.1, R99.2
- new net: C280.1, U29.7 (DVDT)
- new net: C279.1, U27.7 (DVDT)
- new net: C312.1, U21.6 (BST)
- new net: C281.2, L15.1, U30.5 (SW)
- new net: C281.1, U30.6 (BST)
- new net BOOT_PWR: C286.1, C287.2, D1.1 (K), D5.1 (K), L16.1
- new net OVLO: R98.1, R99.1, U27.2 (OVLO)
- new net PWR_3V3D_EN: U21.2 (EN)
- new net PWR_MAIN_EN: R97.1, U27.1 (EN/UVLO)
- new net PWR_MAIN_IMON: U27.9 (IMON)
- new net PWR_MAIN_PG: U27.3 (PG)
- new net PWR_MP_EN: R96.1, U29.1 (EN/UVLO)
- new net PWR_MP_IMON: U29.9 (IMON)
- new net PWR_MP_PG: U29.3 (PG)
- new net SR_C0: C284.1, C285.1, L16.2, U30.2 (EN), U30.3 (IN)
- new net VDD_3V3D: JP14.2 (B)
- new net VDD_MCU: JP13.2 (B)
- new net VDD_SYSTEM: U29.6 (OUT)
Other:
- sheet TPS5430DD_DCDC ports: added none; removed FB_GND, GND
- sheet TPS5430DD_DCDC1 ports: added none; removed FB_GND, GND
- company: (none) -> Tronex s.r.o. / Tronex Group USA LLC
- title: (none) -> TRNX SDR Carrier board
- moved on the sheet: D2, J21, J22, JP10, JP11, JP12, JP9, R2, R3, R93, R94
