File: TRX055.01.01.PB.00.00/RF_If.kicad_sch (KiCad schematic)
At the start: 8 parts, among them J11 HYCW12-SMAW0863-1365B, J12 U.FL-R-SMT-1(80), J13 HYCW12-SMAW0863-1365B, J14 U.FL-R-SMT-1(80), J15 HYCW12-SMAW0863-1365B, J16 U.FL-R-SMT-1(80), J17 HYCW12-SMAW0863-1365B, J18 U.FL-R-SMT-1(80)

Commit message: V0.1 - production, added brig-up comments
Other:
- company: (none) -> Tronex s.r.o. / Tronex Group USA LLC
- title: (none) -> TRNX SDR Carrier board
Changed lines of the file:
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@@
 	(generator_version "9.0")
 	(paper "A4")
+	(title_block
+		(title "TRNX SDR Carrier board")
+		(date "2025-11-18")
+		(rev "0.1")
+		(company "Tronex s.r.o. / Tronex Group USA LLC")
+	)
 	(wire
 		(pts
