File: TRX055.01.01.PB.00.00/System_Managament.kicad_sch (KiCad schematic)
At the start: 18 parts, among them U17 STM32G070RBTx, U18 TL431DBZ, Y2 X322525MOB4SI, Y3 XKXGI-SUA-32.768K

Commit message: V0.1 - production, added brig-up comments
Parts:
- removed C178: M1, Capacitor_SMD:C_0201_0603Metric, symbol PPA-Pasive:Cap
- added C294, C295, C296, C297, C298, C299, C300, C301, C302, C303, C304, C305, C306, C307: M1, Capacitor_SMD:C_0201_0603Metric, symbol PPA-Pasive:Cap
- added C323: 10M, Capacitor_SMD:C_0603_1608Metric, symbol PPA-Pasive:Cap
- added R110, R111, R112, R113, R114, R115, R116, R117, R118, R119, R120, R121, R122, R123, R124, R125, R126, R127, R128, R130, R131, R132, R133, R134, R135, R136, R143: 10K, Resistor_SMD:R_0402_1005Metric, symbol PPA-Pasive:Res
- added R129: 100K, Resistor_SMD:R_0402_1005Metric, symbol PPA-Pasive:Res
- R86: value 33R -> 10K
Connections:
- net I2C2_A_SCL is gone; now on net I2C2_C_SCL: U17.43 (PA11/PA9)
- net I2C2_A_SDA is gone; now on net I2C2_C_SDA: U17.44 (PA12/PA10)
- net ADC1_IN0: now also C295.1, R111.2, R112.1
- net ADC1_IN1: now also C296.1, R113.2, R114.1
- net ADC1_IN10: now also C305.1, R131.2, R132.1
- net ADC1_IN2: now also C297.1, R115.2, R116.1
- net ADC1_IN3: now also C298.1, R117.2, R118.1
- net ADC1_IN4: now also C299.1, R119.2, R120.1
- net ADC1_IN5: now also C300.1, R121.2, R122.1
- net ADC1_IN6: now also C301.1, R123.2, R124.1
- net ADC1_IN7: now also C302.1, R125.2, R126.1
- net ADC1_IN8: now also C303.1, R127.2, R128.1
- net ADC1_IN9: now also C304.1, R129.2, R130.1
- net GND: now also C294.2, C295.2, C296.2, C297.2, C298.2, C299.2, C300.2, C301.2, C302.2, C303.2, C304.2, C305.2, C306.2, C307.2, C323.2, R112.2, R114.2, R116.2, R118.2, R120.2, R122.2, R124.2, R126.2, R128.2, R130.2, R132.2, R134.2, R136.2
- net I2C1_A_SCL: now also U17.60 (PB6); no longer U17.37 (PA9/NC)
- net I2C1_A_SDA: now also U17.61 (PB7); no longer U17.42 (PA10/NC)
- net I2C2_C_SCL: no longer U17.30 (PB10)
- net I2C2_C_SDA: no longer U17.31 (PB11)
- net VREF: now also C323.1
- net VDD_MCU: now reaches FB16.1
- net VDD_MCU: now also R110.1, R143.1
- net at C179.1, U17.6 (VBAT): now also R143.2
- net DBG_SMU_NRST: now reaches U17.12 (NRST)
- net DBG_SMU_NRST: now also C294.1, R110.2
- net GPIO5: now reaches U17.13 (PC0)
- net GPIO6: now reaches U17.14 (PC1)
- net GPIO7: now reaches U17.15 (PC2)
- net GPIO8: now reaches U17.16 (PC3)
- net GPIO0: now reaches U17.2 (PC12)
- net GPIO9: now reaches U17.3 (PC13)
- net ADCIN16: now reaches U17.32 (PB12)
- net GPIO12: now reaches U17.35 (PB15)
- net GPIO16: now reaches U17.39 (PC7)
- net GPIO18: now reaches U17.41 (PD9)
- net GPIO11: now reaches U17.47 (PA15)
- net GPIO4: now reaches U17.48 (PC8)
- net GPIO3: now reaches U17.49 (PC9)
- net SPI2_NSS: now reaches U17.50 (PD0)
- net SPI2_SCK: now reaches U17.51 (PD1)
- net GPIO10: now reaches U17.52 (PD2)
- net SPI2_MISO: now reaches U17.53 (PD3)
- net SPI2_MOSI: now reaches U17.54 (PD4)
- net GPIO2: now reaches U17.58 (PB4)
- net GPIO1: now reaches U17.59 (PB5)
- net I2C2_B_SCL renamed GPIO14
- net I2C2_B_SDA renamed GPIO13
- net SWCLK renamed DBG_SMU_SWCLK
- net SWDIO renamed DBG_SMU_SWDIO
- net USART1_RX renamed ADCIN17
- net USART1_TX renamed ADCIN18
- net USART3_RX renamed DBG_UART_SMU_RX
- net USART3_TX renamed DBG_UART_SMU_TX
- new net ADC1_IN11: C306.1, R133.2, R134.1, U17.30 (PB10)
- new net ADC1_IN15: C307.1, R135.2, R136.1, U17.31 (PB11)
- new net GPIO15: U17.42 (PA10/NC)
- new net PWR_CORE: R127.1
- new net SR_A0: R117.1
- new net SR_A1: R111.1
- new net SR_A2: R123.1
- new net SR_A3: R125.1
- new net SR_B0: R119.1
- new net SR_B1: R121.1
- new net SR_B2: R115.1
- new net SR_B3: R113.1
- new net SR_C0: R131.1
- new net VDD_3V3D: R135.1
- new net VDD_5V5A: R133.1
- new net VDD_MAIN_PWR: R129.1
Other:
- company: (none) -> Tronex s.r.o. / Tronex Group USA LLC
- title: (none) -> TRNX SDR Carrier board
- moved on the sheet: C174, C175, C176, C177, C179, C180, C181, C182, C183, FB16, FB17, R86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
