File: TRX055.01.01.PB.00.00/TPS5430DD_DCDC.kicad_sch (KiCad schematic)
At the start: 16 parts, among them U7 TPS54531DDAR

Commit message: V0.1 - production, added brig-up comments
Parts:
- renumbered L14 to L13
Connections:
- net PGND1 renamed GND
Other:
- company: (none) -> Tronex s.r.o. / Tronex Group USA LLC
- title: (none) -> TRNX SDR Carrier board
