File: TRX055.01.01.PB.00.00/TRX055.01.01.PB.00.00.kicad_sch (KiCad schematic)
At the start: 23 parts, among them U1 XC7Z015-1CLG485I, U10 PI7C9X2G608ELBZXAE

Commit message: Update Layout
Parts:
- removed C100, C101, C102, C103, C104, C105, C106, C107, C88, C89, C90, C91, C92, C93, C94, C95, C96, C97, C98, C99: M1, Capacitor_SMD:C_0201_0603Metric, symbol PPA-Pasive:Cap
- removed unit 1 of U1
- removed U10: PI7C9X2G608ELBZXAE, PI7C9X2G608ELBZXAE:XCVR_PI7C9X2G608ELBZXAE, symbol PI7C9X2G608ELBZXAE:PI7C9X2G608ELBZXAE
- added unit 11 of U1
- added U13: XC7Z015-1CLG485I, CLG485XC7Z012S/XC7Z015_AMD, symbol XC7Z015-1CLG485C:XC7Z015-1CLG485I
- FL1: footprint ppa-forms:module_srd_kit -> Inductor_THT:Choke_Schaffner_RN102-04-14.0x14.0mm
- U1: footprint XC7Z015:CLG485XC7Z012S&slash_XC7Z015_AMD -> CLG485XC7Z012S/XC7Z015_AMD; JLCPCB Part # (none) -> C1522056
Other:
- added sheet ETH_PHY_Metal (ETH_PHY_Metal.kicad_sch)
- added sheet SFP_Port (SFP.kicad_sch)
- added sheet ZYNQ_Bank_112 (ZYNQ_Bank_112.kicad_sch)
- added sheet ZynqConfig (ZynqConfig.kicad_sch)

Commit message: V0.2
Connections:
- net A1_HS_4_P: now reaches U1.AA11 (IO_L7P_T1_13)
- net A1_HS_6_P: now reaches U1.AA12 (IO_L8P_T1_13)
- net A1_HS_11_P: now reaches U1.AA14 (IO_L11P_T1_SRCC_13)
- net A1_HS_11_N: now reaches U1.AA15 (IO_L11N_T1_SRCC_13)
- net A1_HS_15_P: now reaches U1.AA16 (IO_L14P_T2_SRCC_13)
- net A1_HS_15_N: now reaches U1.AA17 (IO_L14N_T2_SRCC_13)
- net A1_HS_4_N: now reaches U1.AB11 (IO_L7N_T1_13)
- net A1_HS_6_N: now reaches U1.AB12 (IO_L8N_T1_13)
- net A1_HS_8_P: now reaches U1.AB13 (IO_L9P_T1_DQS_13)
- net A1_HS_8_N: now reaches U1.AB14 (IO_L9N_T1_DQS_13)
- net A1_HS_13_P: now reaches U1.AB16 (IO_L17P_T2_13)
- net A1_HS_13_N: now reaches U1.AB17 (IO_L17N_T2_13)
- net A1_HS_5_P: now reaches U1.V11 (IO_L4P_T0_13)
- net A1_HS_12_P: now reaches U1.V15 (IO_L2P_T0_13)
- net A1_HS_14_P: now reaches U1.V16 (IO_L23P_T3_13)
- net A1_HS_5_N: now reaches U1.W11 (IO_L4N_T0_13)
- net A1_HS_9_P: now reaches U1.W12 (IO_L3P_T0_DQS_13)
- net A1_HS_9_N: now reaches U1.W13 (IO_L3N_T0_DQS_13)
- net A1_HS_12_N: now reaches U1.W15 (IO_L2N_T0_13)
- net A1_HS_14_N: now reaches U1.W16 (IO_L23N_T3_13)
- net A1_HS_10_P: now reaches U1.Y12 (IO_L10P_T1_13)
- net A1_HS_10_N: now reaches U1.Y13 (IO_L10N_T1_13)
Other:
- moved on the sheet: FL1, U1B

Commit message: +ETH +USB +Connectors
Parts:
- removed FL1: Choke_Schaffner_RN102-0.3-02-12M, Inductor_THT:Choke_Schaffner_RN102-04-14.0x14.0mm, symbol Filter:Choke_Schaffner_RN102-0.3-02-12M
Connections:
- net TMDS_D0_P: now reaches U1.A4 (IO_L10N_T1_AD11N_35)
- net TMDS_D0_N: now reaches U1.A5 (IO_L10P_T1_AD11P_35)
- net TMDS_CLK_P: now reaches U1.A6 (IO_L9N_T1_DQS_AD3N_35)
- net TMDS_CLK_N: now reaches U1.A7 (IO_L9P_T1_DQS_AD3P_35)
- net TMDS_D2_P: now reaches U1.B3 (IO_L13N_T2_MRCC_35)
- net TMDS_D2_N: now reaches U1.B4 (IO_L13P_T2_MRCC_35)
- net TMDS_D1_P: now reaches U1.E5 (IO_L5N_T0_AD9N_35)
- net TMDS_D1_N: now reaches U1.F5 (IO_L5P_T0_AD9P_35)
Other:
- added sheet HDMI (hdmi.kicad_sch)
- added sheet USB_C (USB_C.kicad_sch)
- sheet ETH_PHY_Metal ports: added RGMII_RX_CLK, RGMII_RX_CTL, RGMII_RX_D0, RGMII_RX_D1, RGMII_RX_D2, RGMII_RX_D3, RGMII_TX_CLK, RGMII_TX_CTL, RGMII_TX_D0, RGMII_TX_D1, RGMII_TX_D2, RGMII_TX_D3, SMI_MDC, SMI_MDIO; removed none
- sheet SFP_Port ports: added SFP_RX_N, SFP_RX_P, SFP_TX_N, SFP_TX_P; removed none
- sheet Zynq_PSMIO ports: added RGMII_RX_CLK, RGMII_RX_CTL, RGMII_RX_D0, RGMII_RX_D1, RGMII_RX_D2, RGMII_RX_D3, RGMII_TX_CLK, RGMII_TX_CTL, RGMII_TX_D0, RGMII_TX_D1, RGMII_TX_D2, RGMII_TX_D3, SMI_MDC, SMI_MDIO, USB_DM, USB_DP; removed none
- note added: "74HC595D,118"

Commit message: + add clocks + add PSU
Parts:
- added FB40: BLM18PG330SN1D, Inductor_SMD:L_0603_1608Metric, symbol Device:FerriteBead
- added U19, U23: TXU0304, Package_DFN_QFN:DHVQFN-14-1EP_2.5x3mm_P0.5mm_EP1x1.5mm, symbol ppa-ic-com:TXU0304QWBQARQ1
- added U22: TCA6408ARSVR, ppa-active:UQFN-16_L2.6-W1.8-P0.40-BL, symbol ppa-ic-com:TCA6408ARSVR
- added U26: FUSB340TMX, ppa-active:TMLP-18_L2.8-W2.0-P0.40-BL-EP, symbol ppa-ic-com:FUSB340TMX
- U1: value XC7Z015-1CLG485I -> XC7Z015-2CLG485I; JLCPCB Part # C1522056 -> C1522056
- U1: renamed from U13; value XC7Z015-1CLG485I -> XC7Z015-2CLG485I; JLCPCB Part # (none) -> C1522056
Connections:
- net A1_HS1_CLK_N: now also U1.AA16 (IO_L14P_T2_SRCC_13)
- net A1_HS1_CLK_P: now also U1.AA17 (IO_L14N_T2_SRCC_13)
- net A1_HS_10_N: now also U1.V15 (IO_L2P_T0_13); no longer U1.Y13 (IO_L10N_T1_13)
- net A1_HS_10_P: now also U1.W15 (IO_L2N_T0_13); no longer U1.Y12 (IO_L10P_T1_13)
- net A1_HS_11_N: now also U1.AA14 (IO_L11P_T1_SRCC_13); no longer U1.AA15 (IO_L11N_T1_SRCC_13)
- net A1_HS_11_P: now also U1.AA15 (IO_L11N_T1_SRCC_13); no longer U1.AA14 (IO_L11P_T1_SRCC_13)
- net A1_HS_12_N: now also U1.V16 (IO_L23P_T3_13); no longer U1.W15 (IO_L2N_T0_13)
- net A1_HS_12_P: now also U1.W16 (IO_L23N_T3_13); no longer U1.V15 (IO_L2P_T0_13)
- net A1_HS_13_N: now also U1.W17 (IO_L24P_T3_13); no longer U1.AB17 (IO_L17N_T2_13)
- net A1_HS_13_P: now also U1.Y17 (IO_L24N_T3_13); no longer U1.AB16 (IO_L17P_T2_13)
- net A1_HS_14_N: now also U1.AB16 (IO_L17P_T2_13); no longer U1.W16 (IO_L23N_T3_13)
- net A1_HS_14_P: now also U1.AB17 (IO_L17N_T2_13); no longer U1.V16 (IO_L23P_T3_13)
- net A1_HS_15_N: now also U1.AB21 (IO_L15P_T2_DQS_13); no longer U1.AA17 (IO_L14N_T2_SRCC_13)
- net A1_HS_15_P: now also U1.AB22 (IO_L15N_T2_DQS_13); no longer U1.AA16 (IO_L14P_T2_SRCC_13)
- net A1_HS_5_N: now also U1.V11 (IO_L4P_T0_13); no longer U1.W11 (IO_L4N_T0_13)
- net A1_HS_5_P: now also U1.W11 (IO_L4N_T0_13); no longer U1.V11 (IO_L4P_T0_13)
- net A1_HS_6_N: now also U1.W12 (IO_L3P_T0_DQS_13); no longer U1.AB12 (IO_L8N_T1_13)
- net A1_HS_6_P: now also U1.W13 (IO_L3N_T0_DQS_13); no longer U1.AA12 (IO_L8P_T1_13)
- net A1_HS_7_N: now also U1.AB12 (IO_L8N_T1_13)
- net A1_HS_7_P: now also U1.AA12 (IO_L8P_T1_13)
- net A1_HS_8_N: now also U1.AB13 (IO_L9P_T1_DQS_13); no longer U1.AB14 (IO_L9N_T1_DQS_13)
- net A1_HS_8_P: now also U1.AB14 (IO_L9N_T1_DQS_13); no longer U1.AB13 (IO_L9P_T1_DQS_13)
- net A1_HS_9_N: now also U1.Y12 (IO_L10P_T1_13); no longer U1.W13 (IO_L3N_T0_DQS_13)
- net A1_HS_9_P: now also U1.Y13 (IO_L10N_T1_13); no longer U1.W12 (IO_L3P_T0_DQS_13)
- net GT_RX0_N: now also U26.5 (SSRXCOM+)
- net GT_RX0_P: now also U26.4 (SSRXCOM-)
- net GT_TX0_N: now also U26.2 (SSTXCOM+)
- net GT_TX0_P: now also U26.1 (SSTXCOM-)
- net Module_A1/MOD_SPI_MISO: now also U19.10 (B4)
- net Module_A1/MOD_SPI_MOSI: now also U19.12 (B2Y)
- net Module_A1/MOD_SPI_SCK: now also U19.13 (B1Y)
- net Module_A3/MOD_SPI_MISO: now also U23.10 (B4)
- net Module_A3/MOD_SPI_MOSI: now also U23.12 (B2Y)
- net Module_A3/MOD_SPI_SCK: now also U23.13 (B1Y)
- net TMDS_D1_N: now also U1.B7 (IO_L8P_T1_AD10P_35); no longer U1.F5 (IO_L5P_T0_AD9P_35)
- net TMDS_D1_P: now also U1.B6 (IO_L8N_T1_AD10N_35); no longer U1.E5 (IO_L5N_T0_AD9N_35)
- net A3_HS_6_P: now reaches U1.A1 (IO_L15N_T2_DQS_AD12N_35)
- net A3_HS_6_N: now reaches U1.A2 (IO_L15P_T2_DQS_AD12P_35)
- net A3_HS_7_N: now reaches U1.B1 (IO_L18N_T2_AD13N_35)
- net A3_HS_7_P: now reaches U1.B2 (IO_L18P_T2_AD13P_35)
- net A3_HS_8_N: now reaches U1.C1 (IO_L16N_T2_35)
- net A3_HS_9_N: now reaches U1.C3 (IO_L14N_T2_AD4N_SRCC_35)
- net A3_HS_4_P: now reaches U1.C4 (IO_L12N_T1_MRCC_35)
- net A3_HS1_CLK_P: now reaches U1.C5 (IO_L11N_T1_SRCC_35)
- net A3_HS1_CLK_N: now reaches U1.C6 (IO_L11P_T1_SRCC_35)
- net A3_HS_8_P: now reaches U1.D1 (IO_L16P_T2_35)
- net A3_HS_10_N: now reaches U1.D2 (IO_L17N_T2_AD5N_35)
- net A3_HS_9_P: now reaches U1.D3 (IO_L14P_T2_AD4P_SRCC_35)
- net A3_HS_4_N: now reaches U1.D5 (IO_L12P_T1_MRCC_35)
- net A3_LS_GPIO_3: now reaches U1.D6 (IO_L2N_T0_AD8N_35)
- net A3_LS_GPIO_2: now reaches U1.D7 (IO_L2P_T0_AD8P_35)
- net A3_HS_10_P: now reaches U1.E2 (IO_L17P_T2_AD5P_35)
- net A3_HS_11_P: now reaches U1.E3 (IO_L21N_T3_DQS_AD14N_35)
- net A3_HS_11_N: now reaches U1.E4 (IO_L21P_T3_DQS_AD14P_35)
- net A3_HS_12_N: now reaches U1.F1 (IO_L23N_T3_35)
- net A3_HS_12_P: now reaches U1.F2 (IO_L23P_T3_35)
- net A3_HS_14_N: now reaches U1.F4 (IO_L20N_T3_AD6N_35)
- net A3_HS_17_P: now reaches U1.F6 (IO_L6N_T0_VREF_35)
- net A3_HS_13_N: now reaches U1.G1 (IO_L24N_T3_AD15N_35)
- net A3_HS_15_N: now reaches U1.G2 (IO_L22N_T3_AD7N_35)
- net A3_HS_15_P: now reaches U1.G3 (IO_L22P_T3_AD7P_35)
- net A3_HS_14_P: now reaches U1.G4 (IO_L20P_T3_AD6P_35)
- net A3_HS_17_N: now reaches U1.G6 (IO_L6P_T0_35)
- net A3_HS_18_P: now reaches U1.G7 (IO_L4N_T0_35)
- net A3_HS_18_N: now reaches U1.G8 (IO_L4P_T0_35)
- net A3_HS_13_P: now reaches U1.H1 (IO_L24P_T3_AD15P_35)
- net A3_HS_16_P: now reaches U1.H3 (IO_L19N_T3_VREF_35)
- net A3_HS_16_N: now reaches U1.H4 (IO_L19P_T3_35)
- net A3_LS_GPIO_1: now reaches U1.H5 (IO_25_35)
- net A3_LS_GPIO_0: now reaches U1.H6 (IO_0_35)
- net A1_HS_17_P: now reaches U1.AA19 (IO_L18P_T2_13)
- net A1_HS_17_N: now reaches U1.AA20 (IO_L18N_T2_13)
- net A1_HS_16_P: now reaches U1.AB18 (IO_L16P_T2_13)
- net A1_HS_16_N: now reaches U1.AB19 (IO_L16N_T2_13)
- net A1_LS_GPIO_2: now reaches U1.T16 (IO_0_13)
- net A1_LS_GPIO_0: now reaches U1.U12 (IO_L5N_T0_13)
- net A1_LS_GPIO_3: now reaches U1.U16 (IO_25_13)
- net A1_HS_18_P: now reaches U1.U19 (IO_L20P_T3_13)
- net A1_LS_GPIO_1: now reaches U1.V14 (IO_L1N_T0_13)
- net A1_HS_18_N: now reaches U1.V19 (IO_L20N_T3_13)
- net SYS_MISO: now reaches U1.J1 (IO_L8N_T1_34)
- net SYS_MISO: now also U19.5 (A4Y), U23.5 (A4Y)
- net SYS_MOSI: now reaches U1.J2 (IO_L8P_T1_34)
- net SYS_MOSI: now also U19.3 (A2), U23.3 (A2)
- net SYS_SCK: now reaches U1.J3 (IO_L9P_T1_DQS_34)
- net SYS_SCK: now also U19.2 (A1), U23.2 (A1)
- net A2_LS_GPIO_0: now reaches U1.J7 (IO_L2P_T0_34)
- net A4_LS_GPIO_0: now reaches U1.K2 (IO_L9N_T1_DQS_34)
- net A3_SPI_EN: now reaches U1.K8 (IO_L1N_T0_34)
- net A3_SPI_EN: now also U23.8 (OE)
- net A4_HS_16_P: now reaches U1.L1 (IO_L10N_T1_34)
- net A4_HS_16_N: now reaches U1.L2 (IO_L10P_T1_34)
- net A4_HS_17_P: now reaches U1.M1 (IO_L15N_T2_DQS_34)
- net A4_HS_17_N: now reaches U1.M2 (IO_L15P_T2_DQS_34)
- net A1_SPI_EN: now reaches U1.M8 (IO_L6P_T0_34)
- net A1_SPI_EN: now also U19.8 (OE)
- net A4_HS_18_P: now reaches U1.N1 (IO_L16P_T2_34)
- net A2_LS_GPIO_2: now reaches U1.N5 (IO_L19N_T3_VREF_34)
- net A2_LS_GPIO_1: now reaches U1.N6 (IO_L19P_T3_34)
- net A4_HS_18_N: now reaches U1.P1 (IO_L16N_T2_34)
- net A2_LS_GPIO_3: now reaches U1.P6 (IO_L20P_T3_34)
- net A2_HS_18_P: now reaches U1.P7 (IO_L24P_T3_34)
- net A2_HS_16_P: now reaches U1.R2 (IO_L17N_T2_34)
- net A2_HS_16_N: now reaches U1.R3 (IO_L17P_T2_34)
- net A2_HS_17_P: now reaches U1.R4 (IO_L23N_T3_34)
- net A2_HS_17_N: now reaches U1.R5 (IO_L23P_T3_34)
- net A2_HS_18_N: now reaches U1.R7 (IO_L24N_T3_34)
- net A4_LS_GPIO_1: now reaches U1.T2 (IO_L13P_T2_MRCC_34)
- net A4_LS_GPIO_2: now reaches U1.U1 (IO_L14N_T2_SRCC_34)
- net A4_LS_GPIO_3: now reaches U1.U2 (IO_L14P_T2_SRCC_34)
- new net: FB40.1, U26.17 (VDD)
- new net +3V3: FB40.2, U22.14 (VCCP), U22.15 (VCCI)
- new net A3_HS_5_N: U1.E5 (IO_L5N_T0_AD9N_35)
- new net A3_HS_5_P: U1.F5 (IO_L5P_T0_AD9P_35)
- new net GND: U19.15 (EP), U19.7 (GND), U22.6 (GND), U23.15 (EP), U23.7 (GND), U26.12 (GND), U26.18 (GND), U26.19 (GND), U26.3 (GND)
- new net SFP_Port/MOD_DEF0: U22.4 (P2)
- new net SFP_Port/MOD_RS: U22.5 (P3)
- new net SFP_Port/MOD_TX_DIS: U22.3 (P1)
- new net SFP_Port/MOD_TX_FAULT: U22.2 (P0)
- new net SFP_Port/SFP_RX_N: U26.10 (SSRX1+)
- new net SFP_Port/SFP_RX_P: U26.11 (SSRX1-)
- new net SFP_Port/SFP_TX_N: U26.16 (SSTX1-)
- new net SFP_Port/SFP_TX_P: U26.15 (SSTX1+)
- new net SYS_I2C_SCL: U22.12 (SCL)
- new net SYS_I2C_SDA: U22.13 (SDA)
- new net USB_RX2_N: U26.8 (SSRX2+)
- new net USB_RX2_P: U26.9 (SSRX2-)
- new net USB_TX2_N: U26.14 (SSTX2-)
- new net USB_TX2_P: U26.13 (SSTX2+)
- new net VCCIO_13: U19.14 (VCCB)
- new net VCCIO_34: U19.1 (VCCA), U23.1 (VCCA)
- new net VCCIO_35: U23.14 (VCCB)
Other:
- added sheet Clocking (board_clocking.kicad_sch)
- added sheet Main_Power (Main_Power.kicad_sch)
- added sheet RF_If (RF_If.kicad_sch)
- added sheet System_Managament (System_Managament.kicad_sch)
- sheet Module_A1 ports: added APP_SPEC_A, APP_SPEC_B, HS_VREF, I2C_SCL, I2C_SDA, LS_GPIO4_HS16_P, LS_GPIO5_HS16_N, LS_GPIO6_HS17_P, LS_GPIO7_HS17_N, LS_GPIO8_HS18_P, LS_GPIO9_HS18_N, LS_VREF; removed LS_GPIO4, LS_GPIO5, LS_GPIO6, LS_GPIO7, LS_GPIO8, LS_GPIO9
- sheet Module_A2 ports: added APP_SPEC_A, APP_SPEC_B, HS_VREF, I2C_SCL, I2C_SDA, LS_GPIO4_HS16_P, LS_GPIO5_HS16_N, LS_GPIO6_HS17_P, LS_GPIO7_HS17_N, LS_GPIO8_HS18_P, LS_GPIO9_HS18_N, LS_VREF; removed LS_GPIO4, LS_GPIO5, LS_GPIO6, LS_GPIO7, LS_GPIO8, LS_GPIO9
- sheet Module_A3 ports: added APP_SPEC_A, APP_SPEC_B, HS_VREF, I2C_SCL, I2C_SDA, LS_GPIO4_HS16_P, LS_GPIO5_HS16_N, LS_GPIO6_HS17_P, LS_GPIO7_HS17_N, LS_GPIO8_HS18_P, LS_GPIO9_HS18_N, LS_VREF; removed LS_GPIO4, LS_GPIO5, LS_GPIO6, LS_GPIO7, LS_GPIO8, LS_GPIO9
- sheet Module_A4 ports: added APP_SPEC_A, APP_SPEC_B, HS_VREF, I2C_SCL, I2C_SDA, LS_GPIO4_HS16_P, LS_GPIO5_HS16_N, LS_GPIO6_HS17_P, LS_GPIO7_HS17_N, LS_GPIO8_HS18_P, LS_GPIO9_HS18_N, LS_VREF; removed LS_GPIO4, LS_GPIO5, LS_GPIO6, LS_GPIO7, LS_GPIO8, LS_GPIO9
- sheet SFP_Port ports: added MOD_DEF0, MOD_DEF1, MOD_DEF2, MOD_RS, MOD_RX_DIS, MOD_TX_DIS, MOD_TX_FAULT; removed none
- sheet USB_C ports: added CLK_N, CLK_P, USBB_DM_N, USBB_DM_P, USB_DM_N, USB_DP_P, USB_HS_RX1_N, USB_HS_RX1_P, USB_HS_RX2_N, USB_HS_RX2_P, USB_HS_TX1_N, USB_HS_TX1_P, USB_HS_TX2_N, USB_HS_TX2_P; removed USB_DM, USB_DP
- sheet ZynqConfig ports: added PS_PCLK, PS_POR, PS_SRST; removed none
- sheet ZynqPower ports: added VCC_CFG, VIN; removed none
- sheet Zynq_PSMIO ports: added REFCLK_I, ULPI_RESET, USB_VBUS; removed none
- note added: "100,125,156.25MHz"
- note added: "24MHz"
- note added: "25MHz"
- moved on the sheet: U1B

Commit message: V0.1 - production, added brig-up comments
Parts:
- added C271, C272, C273, C274, C290, C291, C292, C293: M1, Capacitor_SMD:C_0201_0603Metric, symbol PPA-Pasive:Cap
- added R109, R157, R158, R95: 10K, Resistor_SMD:R_0402_1005Metric, symbol PPA-Pasive:Res
- added U32, U33: TXU0304, Package_DFN_QFN:DHVQFN-14-1EP_2.5x3mm_P0.5mm_EP1x1.5mm, symbol ppa-ic-com:TXU0304QWBQARQ1
- U1: footprint CLG485XC7Z012S/XC7Z015_AMD -> XC7Z015:CLG485XC7Z012S&slash_XC7Z015_AMD
Connections:
- net +3V3: now also C273.1, R95.1
- net A1_HS1_CLK_N: now also U1.AA14 (IO_L11P_T1_SRCC_13); no longer U1.AA16 (IO_L14P_T2_SRCC_13)
- net A1_HS1_CLK_P: now also U1.AA15 (IO_L11N_T1_SRCC_13); no longer U1.AA17 (IO_L14N_T2_SRCC_13)
- net A1_HS_11_N: now also U1.AA17 (IO_L14N_T2_SRCC_13); no longer U1.AA14 (IO_L11P_T1_SRCC_13)
- net A1_HS_11_P: now also U1.AA16 (IO_L14P_T2_SRCC_13); no longer U1.AA15 (IO_L11N_T1_SRCC_13)
- net A1_HS_4_N: now also U1.AA11 (IO_L7P_T1_13); no longer U1.AB11 (IO_L7N_T1_13)
- net A1_HS_4_P: now also U1.AB11 (IO_L7N_T1_13); no longer U1.AA11 (IO_L7P_T1_13)
- net GND: now also U19.4 (A3), U23.4 (A3), U26.7 (OE#), C271.2, C272.2, C273.2, C274.2, C290.2, C291.2, C292.2, C293.2, U32.15 (EP), U32.4 (A3), U32.7 (GND), U33.15 (EP), U33.7 (GND)
- net SFP_Port/MOD_RX_DIS: now also U22.7 (P4)
- net SYS_MISO: now also U32.5 (A4Y)
- net SYS_MOSI: now also U32.2 (A1)
- net SYS_SCK: now also U32.3 (A2)
- net VCCIO_34: now also C290.1, U32.1 (VCCA)
- net at FB40.1, U26.17 (VDD): now also C271.1, C272.1
- net GT_LANE0_SEL: now reaches U26.6 (S)
- net SMU_CS: now reaches U1.J6 (IO_L2N_T0_34)
- net SMU_CS: now also U32.8 (OE)
- net FPGA_CLK_REF_1_N: now reaches U1.K3 (IO_L11N_T1_SRCC_34)
- net FPGA_CLK_REF_1_P: now reaches U1.K4 (IO_L11P_T1_SRCC_34)
- net EXTIO_CS: now reaches U1.K5 (IO_L7N_T1_34)
- net EXTIO_CLK_N: now reaches U1.L4 (IO_L12N_T1_MRCC_34)
- net EXTIO_CLK_P: now reaches U1.L5 (IO_L12P_T1_MRCC_34)
- net EXTIO_D0_N: now reaches U1.N3 (IO_L21N_T3_DQS_34)
- net EXTIO_D0_P: now reaches U1.N4 (IO_L21P_T3_DQS_34)
- net EXTIO_D1_N: now reaches U1.P2 (IO_L18N_T2_34)
- net EXTIO_D1_P: now reaches U1.P3 (IO_L18P_T2_34)
- net FPGA_CLK_REF_0: now reaches U1.T1 (IO_L13N_T2_MRCC_34)
- net at U22.1 (RESET#): now also C274.1, R95.2
- net USB_SW_S2: now reaches U22.10 (P7)
- net USB_SW_S1: now reaches U22.8 (P5)
- net USB_SW_S2_OE: now reaches U22.9 (P6)
- new net +1V8: C293.1, R157.1, R158.1, U33.14 (VCCB), U33.8 (OE)
- new net PS_UART1_RX: U33.11 (B3Y)
- new net PS_UART1_TX: U33.10 (B4)
- new net SMU/GPIO3: R157.2
- new net SMU/GPIO4: R158.2
- new net SMU/SPI2_MISO: U32.10 (B4)
- new net SMU/SPI2_MOSI: U32.13 (B1Y)
- new net SMU/SPI2_NSS: R109.2, U32.11 (B3Y)
- new net SMU/SPI2_SCK: U32.12 (B2Y)
- new net SMU/USART2_RX: U33.5 (A4Y)
- new net SMU/USART2_TX: U33.4 (A3)
- new net VDD_MCU: C291.1, C292.1, R109.1, U32.14 (VCCB), U33.1 (VCCA)
Other:
- sheet System_Managament renamed SMU
- added sheet External_Interface (ExtInt.kicad_sch)
- sheet Clocking ports: added EXT_REF_EN; removed none
- sheet HDMI ports: added HDMI_HPD, HDMI_SCL, HDMI_SDA; removed none
- sheet Main_Power ports: added PWR_3V3D_EN, PWR_5V5A_EN, PWR_CORE, PWR_CORE_EN, PWR_MAIN_EN, PWR_MAIN_IMON, PWR_MAIN_PG, PWR_MP_EN, PWR_MP_IMON, PWR_MP_PG, VDD_SYSTEM; removed none
- sheet SMU ports: added ADCIN16, ADCIN17, ADCIN18, DBG_SMU_NRST, DBG_SMU_SWCLK, DBG_SMU_SWDIO, DBG_UART_SMU_RX, DBG_UART_SMU_TX, GPIO0, GPIO1, GPIO10, GPIO11, GPIO12, GPIO13, GPIO14, GPIO15, GPIO16, GPIO17, GPIO18, GPIO2, GPIO3, GPIO4, GPIO5, GPIO6, GPIO7, GPIO8, GPIO9, SPI2_MISO, SPI2_MOSI, SPI2_NSS, SPI2_SCK, USART2_RX, USART2_TX; removed I2C2_A_SCL, I2C2_A_SDA, I2C2_B_SCL, I2C2_B_SDA
- sheet USB_C ports: added USB_CC_SCL, USB_CC_SDA, USB_SW_S1, USB_SW_S2, USB_SW_S2_OE, USB_VBUS; removed none
- sheet ZynqConfig ports: added DBG_SMU_NRST, DBG_SMU_SWCLK, DBG_SMU_SWDIO, DBG_UART_RX, DBG_UART_SMU_RX, DBG_UART_SMU_TX, DBG_UART_TX, VCC_CFG; removed none
- sheet ZynqPower ports: added RAIL_10_EN; removed none
- sheet Zynq_PSMIO ports: added PS_UART0_RX, PS_UART0_TX, PS_UART1_RX, PS_UART1_TX; removed none
- note added: "BUG_01 - missing power connection for Clocking circuits"
- note added: "BUG_02 - Calculate power source feedback dividers"
- note added: "BUG_03 - SMU MCU - check divider for voltage senses from 20V rails"
- note added: "BUG_04 - Ethernet - Eth magnetics connection - disconnect TAB"
- note added: "BUG_05 - Duplicated GTX coupling caps"
- note added: "BUG_06 - I2C SDA/SCL swaped. Run in bit-bang mode"
- note removed: "SI5351B-B02073-GM"
- note removed: "TPS6521903RHBR (C18716455)"
- company: (none) -> Tronex s.r.o. / Tronex Group USA LLC
- title: (none) -> TRNX SDR Carrier board
- moved on the sheet: FB40, U1B, U22, U26
