File: TRX055.01.01.PB.00.00/board_clocking.kicad_sch (KiCad schematic)
At the start: 35 parts, among them J19 Conn_Coaxial, J20 Conn_Coaxial, U13 5P35023B-000NLGI, U16 5P35023B-000NLGI

Commit message: V0.1 - production, added brig-up comments
Parts:
- added C308, C309, C315, C316, C317, C318, C319, C320, C321, C322, C382, C383: M1, Capacitor_SMD:C_0201_0603Metric, symbol PPA-Pasive:Cap
- added FB41, FB42, FB43, FB44, FB45: GZ1005U102TF, Inductor_SMD:L_0402_1005Metric_Pad0.77x0.64mm_HandSolder, symbol Device:FerriteBead
- added R141, R163: 33R, Resistor_SMD:R_0402_1005Metric, symbol PPA-Pasive:Res
- added R142, R164, R165, R166: 10K, Resistor_SMD:R_0402_1005Metric, symbol PPA-Pasive:Res
- added U28: SN74LVC1G125DCKR, Package_TO_SOT_SMD:SOT-353_SC-70-5, symbol 74xGxx:74LVC1G125
Connections:
- net CLK_PWR: now also R142.1
- net CLK_PWR_VBAT: now also R142.2
- net GND: now also C308.2, C309.2, C315.2, C316.2, C317.2, C318.2, C319.2, C320.2, C321.2, C322.2, C383.1, R164.2, U28.3 (GND)
- net at J19.1 (In): now also R85.2
- net VDD_DIFF: now reaches U16.11 (VDDSE2)
- net VDD_DIFF: now also U13.16 (VDDDIFF1), U13.22 (VDDDIFF2), U16.16 (VDDDIFF1), U16.22 (VDDDIFF2), C308.1, C309.1, C315.1, C316.1, C322.1, C383.2, FB42.1, R165.1, R166.1, U28.5 (VCC)
- net VDD_18F: now reaches U16.13 (VDDSE1)
- net VDD_18F: now also C318.1, FB43.1
- net VDD_34F: now reaches U16.20 (VDDSE3)
- net VDD_34F: now also U13.13 (VDDSE1), C317.1, C320.1, FB41.1
- net at J20.1 (In): now also R141.1; no longer R85.2
- net VDD_35F: now reaches U13.11 (VDDSE2)
- net VDD_35F: now also C321.1, FB45.1
- net VDD_13F: now reaches U13.20 (VDDSE3)
- net VDD_13F: now also C319.1, FB44.1
- net SE_A_REF_O: now reaches R77.2, U13.5 (CLKINB/X1)
- net SE_A_REF_O: now also R163.2
- new net: C382.2, R164.1, R165.2, U28.2
- new net: C382.1, R141.2
- new net: R163.1, U28.4
- new net +1V8: FB43.2
- new net +3V3: FB42.2
- new net EXT_REF_EN: R166.2, U28.1
- new net VCCIO_13: FB44.2
- new net VCCIO_34: FB41.2
- new net VCCIO_35: FB45.2
Other:
- company: (none) -> Tronex s.r.o. / Tronex Group USA LLC
- title: (none) -> TRNX SDR Carrier board
- moved on the sheet: C167, C168, C172, C173, J19, J20, R22, R23, R24, R25, R74, R75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
