File: TRX055.01.01.PB.00.00/hdmi.kicad_sch (KiCad schematic)
At the start: 1 part, among them J7 HDMI_D_1.4

Commit message: + add clocks + add PSU
Parts:
- J7: JLCPCB Part # (none) -> C563878
Changed lines of the file:
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@@
+			)
+		)
+		(property "LCSC Part Name" ""
+			(at 198.12 88.9 0)
+			(effects
+				(font
+					(size 1.27 1.27)
+				)
+				(hide yes)
+			)
+		)
+		(property "Manufacturer" ""
+			(at 198.12 88.9 0)
+			(effects
+				(font
+					(size 1.27 1.27)
+				)
+				(hide yes)
+			)
+		)
+		(property "Manufacturer Part" ""
+			(at 198.12 88.9 0)
+			(effects
+				(font
+					(size 1.27 1.27)
+				)
+				(hide yes)
+			)
+		)
+		(property "Supplier" ""
+			(at 198.12 88.9 0)
+			(effects
+				(font
+					(size 1.27 1.27)
+				)
+				(hide yes)
+			)
+		)
+		(property "Supplier Part" ""
+			(at 198.12 88.9 0)
+			(effects
+				(font
+					(size 1.27 1.27)
+				)
+				(hide yes)
+			)
+		)
+		(property "JLCPCB Part #" "C563878"
+			(at 198.12 88.9 0)
+			(effects
+				(font
+					(size 1.27 1.27)
+				)
+				(hide yes)
 			)
 		)

Commit message: V0.1 - production, added brig-up comments
Parts:
- added Q1, Q2, Q3: NTS4001NT1G, Package_TO_SOT_SMD:SOT-323_SC-70, symbol Transistor_FET:BSS138
- added R101, R102, R103, R104, R105, R106: 10K, Resistor_SMD:R_0402_1005Metric, symbol PPA-Pasive:Res
Connections:
- net GND: now also J7.SH
- net at J7.1 (HPD/HEAC-): now also Q3.3 (D), R105.2
- net at J7.17 (SCL): now also Q1.3 (D), R101.2
- net at J7.18 (SDA): now also Q2.3 (D), R102.2
- net VDD_5V5A: now reaches J7.19 (+5V)
- net VDD_5V5A: now also R101.1, R102.1, R105.1
- new net +3V3: Q1.1 (G), Q2.1 (G), Q3.1 (G), R103.1, R104.1, R106.1
- new net HDMI_HPD: Q3.2 (S), R106.2
- new net HDMI_SCL: Q1.2 (S), R103.2
- new net HDMI_SDA: Q2.2 (S), R104.2
Other:
- company: (none) -> Tronex s.r.o. / Tronex Group USA LLC
- title: (none) -> TRNX SDR Carrier board
- moved on the sheet: J7
